File: _saved_DipsyBoard.sch (KiCad schematic (older format))
At the start: 30 parts, among them CON1 SDMMC_Card, P1 USB_OTG, P2 CONN_01X19, P3 CONN_01X19, P6 JTAG, SW1 SW_PUSH, U1 STM32L486Rx-LQFP64, U3 TPS56x200, U4 PUSBMxX4, X1 XTAL

Commit message: push everything to repo
Parts:
- added C? (x2): 22uF, Capacitors_SMD:C_0805, symbol C
- added L?: 470nF, symbol L_Small
- added R? (x5): 10k, symbol R_Small
- D1: footprint (none) -> LEDs:LED-0805
- R3: footprint (none) -> Resistors_SMD:R_0603
Connections:
- net GND: now also C?.2, C?.2, R?.2
- net SDMMC_CMD: now also R?.1
- net SDMMC_D0: now also R?.2
- net SDMMC_D1: now also R?.2
- net SDMMC_D2: now also R?.2
- net SDMMC_D3: now also R?.2
- net VDD: now also L?.2, R?.1, R?.1, R?.1, R?.1; no longer CON1.4 (VDD)
- new net: C?.1, C?.1, CON1.4 (VDD), L?.1
Other:
- moved on the sheet: CON1
