File: BetsyBoard.sch (KiCad schematic (older format))
At the start: 44 parts, among them CON1 SDMMC_Card, P1 USB_OTG, P2 Analog, P3 Digital, P4 JLINK-SWD, P5 POWER, P6 CORTEX-JTAG, SW1 SW_PUSH, U1 STM32L486Rx-LQFP64, U2 TPS63051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

Commit message: Latest
Parts:
- added C15: 0.1uF, smd:SM0603, symbol C
- added P7: PG, xess:HDR_1x1, symbol CONN_01X01
- L2: value 470nH -> 0.47uH; footprint smd:SM0603 -> w_smd_cap:c_1210
- P2, P3: footprint Pin_Headers:Pin_Header_Straight_1x16 -> w_pin_strip:pin_strip_16
- P4: footprint xess:HDR_1x6 -> w_pin_strip:pin_strip_6
- P5: footprint w_pin_strip:pin_socket_2 -> engstad:pin-socket-2
- P6: footprint engstad:smt-pin-header-02x05-127 -> engstad:conn-jtag-0.05
- U1: symbol STM32L486Rx-LQFP64 -> STM32L486Rx-LQFP64-RESCUE-BetsyBoard
Connections:
- net BOOT0: now also R4.1; no longer JP1.2
- net GND: now also JP1.1, P5.2 (P2), C15.2; no longer P5.1 (P1), R4.2
- net OTG_5V: now also P5.1 (P1); no longer P5.2 (P2)
- net PG: now also P7.1 (P1)
- net VDD: now also C15.1; no longer C18.1, U1.1 (VBAT)
- net VDD_SD: now reaches C12.1, C13.1, CON1.4 (VDD), L2.1
- net FB: now reaches R1.2, R2.1, U2.D2 (FB)
- new net: JP1.2, R4.2
- new net VBAT: C18.1, U1.1 (VBAT)
Other:
- note removed: "JTCK/SWCLK: (PA14) Morpho Pin 15 (Row 8L)\nJTMS/SWDIO: (PA13) Morpho Pin 13 (Row 3L)\n~RST~: Arduino pin\n\n"
- moved on the sheet: C18, P4, R4
Changed lines of the file:
@@
 EESchema Schematic File Version 2
+LIBS:BetsyBoard-rescue
 LIBS:power
 LIBS:device
@@
 $EndDescr
 $Comp
-L STM32L486Rx-LQFP64 U1
+L STM32L486Rx-LQFP64-RESCUE-BetsyBoard U1
 U 1 1 55F9D79E
 P 7500 4650
@@
 	6150 3700 6150 4050
 Wire Wire Line
-	700  7000 4350 7000
+	700  7000 2950 7000
 Wire Wire Line
 	1100 7000 1100 7100
@@
 	1100 7500 1100 7400
 Wire Wire Line
-	700  7500 4150 7500
+	700  7500 2950 7500
 Wire Wire Line
 	1450 7500 1450 7400
@@
 	850  7500 850  7600
 Connection ~ 850  7500
-Connection ~ 2950 7000
-Connection ~ 2950 7500
 Wire Wire Line
 	4850 4800 4850 4250
@@
 Text Label 10350 4200 0    60   ~ 0
 ~RST
-Wire Wire Line
-	4150 7500 4150 7400
-Wire Wire Line
-	4150 7100 4150 7000
-Connection ~ 4150 7000
 $Comp
 L C C18
 U 1 1 5603811A
-P 4150 7250
-F 0 "C18" H 4175 7350 50  0000 L CNN
-F 1 "0.1uF" H 4175 7150 50  0000 L CNN
-F 2 "smd:SM0603" H 4188 7100 30  0001 C CNN
-F 3 "" H 4150 7250 60  0000 C CNN
-	1    4150 7250
+P 4900 3000
+F 0 "C18" H 4925 3100 50  0000 L CNN
+F 1 "0.1uF" H 4925 2900 50  0000 L CNN
+F 2 "smd:SM0603" H 4938 2850 30  0001 C CNN
+F 3 "" H 4900 3000 60  0000 C CNN
+	1    4900 3000
 	1    0    0    -1
 $EndComp
@@
 F 0 "P6" H 10100 4300 50  0000 C CNN
 F 1 "CORTEX-JTAG" H 10100 3700 50  0000 C CNN
-F 2 "engstad:smt-pin-header-02x05-127" H 10100 2800 60  0001 C CNN
+F 2 "engstad:conn-jtag-0.05" H 10100 2800 60  0001 C CNN
 F 3 "" H 10100 2800 60  0000 C CNN
 	1    10100 4000
 	1    0    0    -1
 $EndComp
-Text Label 9850 3800 2    60   ~ 0
-VDD
-Text Label 9850 3900 2    60   ~ 0
-GND
-Text Label 9850 4000 2    60   ~ 0
-GND
-Text Label 9850 4200 2    60   ~ 0
-GND
-Text Label 6450 3200 2    60   ~ 0
+Text Label 9300 3800 2    60   ~ 0
 VDD
 Wire Wire Line
@@
 P 3600 5550
 F 0 "L2" H 3630 5590 50  0000 L CNN
-F 1 "470nH" H 3630 5510 50  0000 L CNN
-F 2 "smd:SM0603" H 3600 5550 60  0001 C CNN
+F 1 "0.47uH" H 3630 5510 50  0000 L CNN
+F 2 "w_smd_cap:c_1210" H 3600 5550 60  0001 C CNN
 F 3 "" H 3600 5550 60  0000 C CNN
 	1    3600 5550
@@
 L R R4
 U 1 1 5629BEEA
-P 1400 4500
-F 0 "R4" V 1480 4500 50  0000 C CNN
-F 1 "10k" V 1400 4500 50  0000 C CNN
-F 2 "smd:SM0603" V 1330 4500 30  0001 C CNN
-F 3 "" H 1400 4500 30  0000 C CNN
-	1    1400 4500
-	1    0    0    -1
+P 1750 4200
+F 0 "R4" V 1830 4200 50  0000 C CNN
+F 1 "10k" V 1750 4200 50  0000 C CNN
+F 2 "smd:SM0603" V 1680 4200 30  0001 C CNN
+F 3 "" H 1750 4200 30  0000 C CNN
+	1    1750 4200
+	0    1    1    0
 $EndComp
 $Comp
 L GND #PWR010
 U 1 1 5629BF5F
-P 1400 4650
-F 0 "#PWR010" H 1400 4400 50  0001 C CNN
-F 1 "GND" H 1400 4500 50  0000 C CNN
-F 2 "" H 1400 4650 60  0000 C CNN
-F 3 "" H 1400 4650 60  0000 C CNN
-	1    1400 4650
-	1    0    0    -1
-$EndComp
-Wire Wire Line
-	1400 4350 1400 4250
-Text Label 1800 4000 0    60   ~ 0
+P 1300 4650
+F 0 "#PWR010" H 1300 4400 50  0001 C CNN
+F 1 "GND" H 1300 4500 50  0000 C CNN
+F 2 "" H 1300 4650 60  0000 C CNN
+F 3 "" H 1300 4650 60  0000 C CNN
+	1    1300 4650
+	1    0    0    -1
+$EndComp
+Text Label 2000 4200 0    60   ~ 0
 BOOT0
-$Comp
-L JUMPER3 JP1
-U 1 1 5629C5E9
-P 1400 4000
-F 0 "JP1" H 1450 3900 50  0000 L CNN
-F 1 "JUMPER3" H 1400 4100 50  0000 C BNN
-F 2 "xess:xess-JP2" H 1400 4250 60  0000 C CNN
-F 3 "" H 1400 4000 60  0000 C CNN
-	1    1400 4000
-	0    -1   -1   0
-$EndComp
-Wire Wire Line
-	1500 4000 1800 4000
-Wire Wire Line
-	1400 3750 1400 3550
+Wire Wire Line
+	1300 3500 1300 3950
 $Comp
 L VDD #PWR011
 U 1 1 5629CAD9
-P 1400 3550
-F 0 "#PWR011" H 1400 3400 50  0001 C CNN
-F 1 "VDD" H 1400 3700 50  0000 C CNN
-F 2 "" H 1400 3550 60  0000 C CNN
-F 3 "" H 1400 3550 60  0000 C CNN
-	1    1400 3550
+P 1300 3500
+F 0 "#PWR011" H 1300 3350 50  0001 C CNN
+F 1 "VDD" H 1300 3650 50  0000 C CNN
+F 2 "" H 1300 3500 60  0000 C CNN
+F 3 "" H 1300 3500 60  0000 C CNN
+	1    1300 3500
 	1    0    0    -1
 $EndComp
@@
 L CONN_01X06 P4
 U 1 1 562A469F
-P 10150 1250
-F 0 "P4" H 10150 1600 50  0000 C CNN
-F 1 "JLINK-SWD" H 10150 900 50  0000 C CNN
-F 2 "xess:HDR_1x6" H 10150 1250 60  0001 C CNN
-F 3 "" H 10150 1250 60  0000 C CNN
-	1    10150 1250
+P 10150 4800
+F 0 "P4" H 10150 5150 50  0000 C CNN
+F 1 "JLINK-SWD" H 10150 4450 50  0000 C CNN
+F 2 "w_pin_strip:pin_strip_6" H 10150 4800 60  0001 C CNN
+F 3 "" H 10150 4800 60  0000 C CNN
+	1    10150 4800
 	-1   0    0    -1
 $EndComp
-Text Label 10350 1200 0    60   ~ 0
-GND
-Text Label 10350 1100 0    60   ~ 0
+Text Label 10350 4650 0    60   ~ 0
 JTCK/SWCLK
-Text Label 10350 1000 0    60   ~ 0
+Text Label 10350 4550 0    60   ~ 0
 VDD
-Text Label 10350 1300 0    60   ~ 0
+Text Label 10350 4850 0    60   ~ 0
 JTMS/SWDIO
-Text Label 10350 1400 0    60   ~ 0
+Text Label 10350 4950 0    60   ~ 0
 ~RST
-Text Notes 9900 5900 0    60   ~ 0
-JTCK/SWCLK: (PA14) Morpho Pin 15 (Row 8L)\nJTMS/SWDIO: (PA13) Morpho Pin 13 (Row 3L)\n~RST~: Arduino pin\n\n
 $Comp
 L PUSBMxX4 U4
@@
 Connection ~ 1950 1900
 Wire Wire Line
-	850  3550 850  3700
+	850  3500 850  3700
 $Comp
 L LED D3
@@
 L VDD #PWR019
 U 1 1 562B52A7
-P 850 3550
-F 0 "#PWR019" H 850 3400 50  0001 C CNN
-F 1 "VDD" H 850 3700 50  0000 C CNN
-F 2 "" H 850 3550 60  0000 C CNN
-F 3 "" H 850 3550 60  0000 C CNN
-	1    850  3550
+P 850 3500
+F 0 "#PWR019" H 850 3350 50  0001 C CNN
+F 1 "VDD" H 850 3650 50  0000 C CNN
+F 2 "" H 850 3500 60  0000 C CNN
+F 3 "" H 850 3500 60  0000 C CNN
+	1    850  3500
 	1    0    0    -1
 $EndComp
@@
 F 0 "P2" H 9650 3450 50  0000 C CNN
 F 1 "Analog" H 9650 1750 50  0000 C CNN
-F 2 "Pin_Headers:Pin_Header_Straight_1x16" H 9650 2600 60  0001 C CNN
+F 2 "w_pin_strip:pin_strip_16" H 9650 2600 60  0001 C CNN
 F 3 "" H 9650 2600 60  0000 C CNN
 	1    9650 2600
@@
 F 0 "P3" H 10850 3450 50  0000 C CNN
 F 1 "Digital" H 10850 1750 50  0000 C CNN
-F 2 "Pin_Headers:Pin_Header_Straight_1x16" H 10850 2600 60  0001 C CNN
+F 2 "w_pin_strip:pin_strip_16" H 10850 2600 60  0001 C CNN
 F 3 "" H 10850 2600 60  0000 C CNN
 	1    10850 2600
 	1    0    0    -1
 $EndComp
-Text Label 10350 1500 0    60   ~ 0
+Text Label 10350 5050 0    60   ~ 0
 JTDO/SWO
 $Comp
@@
 F 0 "P5" H 900 1000 50  0000 C CNN
 F 1 "POWER" V 1000 850 50  0000 C CNN
-F 2 "w_pin_strip:pin_socket_2" H 900 850 60  0001 C CNN
+F 2 "engstad:pin-socket-2" H 900 850 60  0001 C CNN
 F 3 "" H 900 850 60  0000 C CNN
 	1    900  850
-	-1   0    0    1
+	-1   0    0    -1
 $EndComp
 Wire Wire Line
@@
 	5750 1050 5750 1150
 Connection ~ 5750 1050
-Wire Wire Line
-	5750 2000 5850 2000
 Connection ~ 5750 1800
-Text Label 5850 2000 0    60   ~ 0
+Text Label 5750 1950 0    60   ~ 0
 PG
 $Comp
@@
 Wire Wire Line
 	5050 1350 5350 1350
+Wire Wire Line
+	2000 4200 1900 4200
+Text Label 10350 4750 0    60   ~ 0
+GND
+$Comp
+L JUMPER3 JP1
+U 1 1 564ECC19
+P 1300 4200
+F 0 "JP1" H 1350 4100 50  0000 L CNN
+F 1 "JUMPER3" H 1300 4300 50  0000 C BNN
+F 2 "xess:xess-JP2" H 1300 4200 60  0001 C CNN
+F 3 "" H 1300 4200 60  0000 C CNN
+	1    1300 4200
+	0    -1   -1   0
+$EndComp
+Wire Wire Line
+	1400 4200 1600 4200
+Wire Wire Line
+	1300 4450 1300 4650
+Text Label 2450 5550 0    60   ~ 0
+VDD_SD
+$Comp
+L CONN_01X01 P7
+U 1 1 564EE352
+P 5750 2200
+F 0 "P7" H 5750 2300 50  0000 C CNN
+F 1 "PG" V 5850 2200 50  0000 C CNN
+F 2 "xess:HDR_1x1" H 5750 2200 60  0001 C CNN
+F 3 "" H 5750 2200 60  0000 C CNN
+	1    5750 2200
+	0    1    1    0
+$EndComp
+$Comp
+L C C15
+U 1 1 564EFD30
+P 9400 4000
+F 0 "C15" H 9425 4100 50  0000 L CNN
+F 1 "0.1uF" H 9425 3900 50  0000 L CNN
+F 2 "smd:SM0603" H 9438 3850 30  0001 C CNN
+F 3 "" H 9400 4000 60  0000 C CNN
+	1    9400 4000
+	1    0    0    -1
+$EndComp
+Wire Wire Line
+	9300 3800 9850 3800
+Wire Wire Line
+	9400 3800 9400 3850
+Connection ~ 9400 3800
+$Comp
+L GND #PWR028
+U 1 1 564F03B1
+P 9600 4350
+F 0 "#PWR028" H 9600 4100 50  0001 C CNN
+F 1 "GND" H 9600 4200 50  0000 C CNN
+F 2 "" H 9600 4350 60  0000 C CNN
+F 3 "" H 9600 4350 60  0000 C CNN
+	1    9600 4350
+	1    0    0    -1
+$EndComp
+Wire Wire Line
+	9850 3900 9750 3900
+Wire Wire Line
+	9750 3900 9750 4200
+Wire Wire Line
+	9750 4000 9850 4000
+Wire Wire Line
+	9400 4200 9850 4200
+Connection ~ 9750 4000
+Wire Wire Line
+	9400 4150 9400 4200
+Wire Wire Line
+	9600 4200 9600 4350
+Connection ~ 9750 4200
+Connection ~ 9600 4200
+$Comp
+L GND #PWR029
+U 1 1 564F36A0
+P 4900 3150
+F 0 "#PWR029" H 4900 2900 50  0001 C CNN
+F 1 "GND" H 4900 3000 50  0000 C CNN
+F 2 "" H 4900 3150 60  0000 C CNN
+F 3 "" H 4900 3150 60  0000 C CNN
+	1    4900 3150
+	1    0    0    -1
+$EndComp
+Wire Wire Line
+	4250 2800 5750 2800
+Wire Wire Line
+	4900 2800 4900 2850
+Wire Wire Line
+	5750 2800 5750 3200
+Wire Wire Line
+	5750 3200 6450 3200
+Connection ~ 4900 2800
+Text Label 4650 1200 0    60   ~ 0
+FB
+Text Label 4250 2800 2    60   ~ 0
+VBAT
 $EndSCHEMATC

Commit message: Newest component
Parts:
- U1: symbol STM32L486Rx-LQFP64-RESCUE-BetsyBoard -> STM32L486Rx-LQFP64
Changed lines of the file:
@@
 EESchema Schematic File Version 2
-LIBS:BetsyBoard-rescue
 LIBS:power
 LIBS:device
@@
 $EndDescr
 $Comp
-L STM32L486Rx-LQFP64-RESCUE-BetsyBoard U1
+L STM32L486Rx-LQFP64 U1
 U 1 1 55F9D79E
 P 7500 4650
-F 0 "U1" H 7500 4650 60  0000 C CNN
-F 1 "STM32L486Rx-LQFP64" H 7500 5125 60  0000 C CNN
+F 0 "U1" H 6800 6400 60  0000 C CNN
+F 1 "STM32L486Rx-LQFP64" H 7500 6400 60  0000 C CNN
 F 2 "Housings_QFP:LQFP-64_10x10mm_Pitch0.5mm" H 7500 4650 60  0001 C CNN
 F 3 "" H 7500 4650 60  0000 C CNN
