File: BetsyBoard.sch (KiCad schematic (older format))
At the start: 50 parts, among them CON1 SDMMC_Card, P1 USB_OTG, P2 Analog, P3 Digital, P4 JLINK-SWD, P5 VIN, P6 CORTEX-JTAG, P7 RTC, P8 BATT, P9 VDD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

Commit message: v0.7
Parts:
- removed C13: 22uF, smd:SM0805, symbol C
- removed CON1: SDMMC_Card, engstad:SCHD3A0100, symbol SDMMC_Card
- removed L2: 0.47uH, smd:SM0603, symbol L_Small
- removed P4: JLINK-SWD, engstad:pin-strip-6, symbol CONN_01X06
- added U5: N25Q00AA, SMD_Packages:SO-16-W, symbol N25Q00AA
- C12: value 22uF -> 0.1uF; footprint smd:SM0805 -> smd:SM0603
- D1, D3: symbol LED -> LED-RESCUE-BetsyBoard
- P1: symbol USB_OTG -> USB_OTG-RESCUE-BetsyBoard
Connections:
- net VDDSD is gone; now on net VDD: C12.1
- net GND: now also U5.10 (VSS)
- net SDMMC_CMD: now also U5.7 (S#)
- net SDMMC_D0: now also U5.15 (DQ0)
- net SDMMC_D1: now also U5.8 (DQ1)
- net SDMMC_D2: now also U5.9 (DQ2/W#/VPP)
- net SDMMC_D3: now also U5.1 (DQ3/HOLD#)
- net VDD: now also U5.2 (VCC)
- net SDMMC_CK renamed SDMMC_CLK
- net SDMMC_CLK: now also U5.16 (C)
Other:
- moved on the sheet: C2, C3, C5, C6, C7, C8

Commit message: More
Parts:
- removed C11: 22uF, smd:SM0805, symbol C
- removed C14: 0.1uF, smd:SM0603, symbol C_Small
- removed L1: 3.3uH, engstad:inductor-smd-1212, symbol INDUCTOR_SMALL
- removed P1: USB_OTG, engstad:usb-micro-b-amphenol-fci-10118194, symbol USB_OTG-RESCUE-BetsyBoard
- removed R1: 33.2k, smd:SM0603, symbol R_Small
- removed R2: 10k, smd:SM0603, symbol R_Small
- removed R6: 10.0k, smd:SM0603, symbol R_Small
- removed U4: TPS56x200, w_smd_trans:sot23-6, symbol TPS56x200
- added J1: USB_OTG, engstad:usb-micro-b-amphenol-fci-10118194, symbol USB_OTG
- added L1: Bead, smd:SM0805, symbol L_Small
- added U4: LP5907MFX, TO_SOT_Packages_SMD:SOT-23-5, symbol LP5907MFX
- C10, C16: value 10uF -> 1uF
- U2: footprint w_smd_trans:sot23-6 -> TO_SOT_Packages_SMD:SOT-23-6
Connections:
- net labels added: VIN
- net labels removed: EN, FB, SW
- wire segments 111 -> 108
Other:
- note removed: "VDD=0.765*(1+R1/R2) = 0.765*4.32=3.3 V\n"
- moved on the sheet: C10, C16, P5, P9, U2
