File: BetsyBoard.sch (KiCad schematic (older format))
At the start: 42 parts, among them J1 USB_OTG, P2 Analog, P3 Digital, P5 VIN, P6 CORTEX-JTAG, P7 RTC, P8 BATT, P9 VDD, SW1 RST, SW2 spdp-2x, U1 STM32L486Rx-LQFP64, U2 RClamp0504S, U3 APX823, U4 LP5907MFX, U5 N25Q00AA, X1 XTAL, Y1 Crystal

Commit message: apx comments
Parts:
- renumbered C10 to C1, C18 to C10, C12 to C11, C2 to C12, C3 to C13, C5 to C14, C6 to C15, C7 to C16, C8 to C17, C16 to C2, C15 to C3, C20 to C4, C4 to C5, C9 to C6, C1 to C7, C17 to C8, C19 to C9, D3 to D2, L3 to L2, P5 to P1, P9 to P2, P6 to P3, P2 to P4, P3 to P5, P8 to P6, R7 to R1, R4 to R2, R5 to R4, SW2 to SW1, SW1 to SW2, U4 to U1, U1 to U4
Other:
- note added: "The APX823's manual reset line (~MR~) \nhas internal pullup of 60 kOhm.\n"
- moved on the sheet: C2
Changed lines of the file:
@@
 $EndDescr
 $Comp
-L STM32L486Rx-LQFP64 U1
+L STM32L486Rx-LQFP64 U4
 U 1 1 55F9D79E
 P 7650 4650
-F 0 "U1" H 6650 6450 60  0000 C CNN
+F 0 "U4" H 6650 6450 60  0000 C CNN
 F 1 "STM32L486Rx-LQFP64" H 7650 6450 60  0000 C CNN
 F 2 "Housings_QFP:LQFP-64_10x10mm_Pitch0.5mm" H 7650 4650 60  0001 C CNN
@@
 VDD
 $Comp
-L C C2
+L C C12
 U 1 1 55FB1A3F
 P 2300 6650
-F 0 "C2" H 2325 6750 50  0000 L CNN
+F 0 "C12" H 2325 6750 50  0000 L CNN
 F 1 "4.7uF" H 2325 6550 50  0000 L CNN
 F 2 "smd:SM0805" H 2338 6500 30  0001 C CNN
@@
 $EndComp
 $Comp
-L C C9
+L C C6
 U 1 1 55FB1A93
 P 5100 2300
-F 0 "C9" H 5125 2400 50  0000 L CNN
+F 0 "C6" H 5125 2400 50  0000 L CNN
 F 1 "0.1uF" H 5125 2200 50  0000 L CNN
 F 2 "smd:SM0603" H 5138 2150 30  0001 C CNN
@@
 $EndComp
 $Comp
-L C C5
+L C C14
 U 1 1 55FB1B14
 P 3250 6650
-F 0 "C5" H 3275 6750 50  0000 L CNN
+F 0 "C14" H 3275 6750 50  0000 L CNN
 F 1 "0.1uF" H 3275 6550 50  0000 L CNN
 F 2 "smd:SM0603" H 3288 6500 30  0001 C CNN
@@
 $EndComp
 $Comp
-L C C6
+L C C15
 U 1 1 55FB1B48
 P 3550 6650
-F 0 "C6" H 3575 6750 50  0000 L CNN
+F 0 "C15" H 3575 6750 50  0000 L CNN
 F 1 "0.1uF" H 3575 6550 50  0000 L CNN
 F 2 "smd:SM0603" H 3588 6500 30  0001 C CNN
@@
 $EndComp
 $Comp
-L C C7
+L C C16
 U 1 1 55FB1BA8
 P 3850 6650
-F 0 "C7" H 3875 6750 50  0000 L CNN
+F 0 "C16" H 3875 6750 50  0000 L CNN
 F 1 "0.1uF" H 3875 6550 50  0000 L CNN
 F 2 "smd:SM0603" H 3888 6500 30  0001 C CNN
@@
 $EndComp
 $Comp
-L C C8
+L C C17
 U 1 1 55FB1BDE
 P 4150 6650
-F 0 "C8" H 4175 6750 50  0000 L CNN
+F 0 "C17" H 4175 6750 50  0000 L CNN
 F 1 "0.1uF" H 4175 6550 50  0000 L CNN
 F 2 "smd:SM0603" H 4188 6500 30  0001 C CNN
@@
 $EndComp
 $Comp
-L C C3
+L C C13
 U 1 1 55FB1E44
 P 2650 6650
-F 0 "C3" H 2675 6750 50  0000 L CNN
+F 0 "C13" H 2675 6750 50  0000 L CNN
 F 1 "1.0uF" H 2675 6550 50  0000 L CNN
 F 2 "smd:SM0603" H 2688 6500 30  0001 C CNN
@@
 $EndComp
 $Comp
-L C C4
+L C C5
 U 1 1 55FB260E
 P 4750 2300
-F 0 "C4" H 4775 2400 50  0000 L CNN
+F 0 "C5" H 4775 2400 50  0000 L CNN
 F 1 "1.0uF" H 4775 2200 50  0000 L CNN
 F 2 "smd:SM0603" H 4788 2150 30  0001 C CNN
@@
 $EndComp
 $Comp
-L C C1
+L C C7
 U 1 1 55FB28C4
 P 10550 3050
-F 0 "C1" V 10500 3100 50  0000 L CNN
+F 0 "C7" V 10500 3100 50  0000 L CNN
 F 1 "0.1uF" V 10600 3100 50  0000 L CNN
 F 2 "smd:SM0603" H 10588 2900 30  0001 C CNN
@@
 JTDO/SWO
 $Comp
-L C C18
+L C C10
 U 1 1 5603811A
 P 4100 4000
-F 0 "C18" H 3900 4100 50  0000 L CNN
+F 0 "C10" H 3900 4100 50  0000 L CNN
 F 1 "0.1uF" H 3850 3900 50  0000 L CNN
 F 2 "smd:SM0603" H 4138 3850 30  0001 C CNN
@@
 $EndComp
 $Comp
-L CONN_02X05 P6
+L CONN_02X05 P3
 U 1 1 56040117
 P 10050 1250
-F 0 "P6" H 10050 1550 50  0000 C CNN
+F 0 "P3" H 10050 1550 50  0000 C CNN
 F 1 "CORTEX-JTAG" H 10050 950 50  0000 C CNN
 F 2 "engstad:conn-jtag-0.05" H 10050 50  60  0001 C CNN
@@
 D16
 $Comp
-L C C10
+L C C1
 U 1 1 560BBDCE
 P 3150 1200
-F 0 "C10" H 3265 1250 50  0000 L CNN
+F 0 "C1" H 3265 1250 50  0000 L CNN
 F 1 "1uF" H 3265 1150 50  0000 L CNN
 F 2 "smd:SM0805" H 3188 1050 30  0001 C CNN
@@
 BOOT0
 $Comp
-L R R4
+L R R2
 U 1 1 5629BEEA
 P 5750 3100
-F 0 "R4" V 5830 3100 50  0000 C CNN
+F 0 "R2" V 5830 3100 50  0000 C CNN
 F 1 "10k" V 5750 3100 50  0000 C CNN
 F 2 "smd:SM0603" V 5680 3100 30  0001 C CNN
@@
 $EndComp
 $Comp
-L L_Small L3
+L L_Small L2
 U 1 1 5629D98A
 P 4500 2100
-F 0 "L3" H 4530 2140 50  0000 L CNN
+F 0 "L2" H 4530 2140 50  0000 L CNN
 F 1 "Bead" H 4530 2060 50  0000 L CNN
 F 2 "smd:SM0805" V 4900 2100 60  0001 C CNN
@@
 $EndComp
 $Comp
-L LED-RESCUE-BetsyBoard D3
+L LED-RESCUE-BetsyBoard D2
 U 1 1 562B4DD6
 P 10550 5350
-F 0 "D3" V 10596 5242 50  0000 R CNN
+F 0 "D2" V 10596 5242 50  0000 R CNN
 F 1 "GREEN" V 10504 5242 50  0000 R CNN
 F 2 "w_smd_leds:Led_0603" H 10550 5350 60  0001 C CNN
@@
 $EndComp
 $Comp
-L R R5
+L R R4
 U 1 1 562B4DDD
 P 10550 5800
-F 0 "R5" H 10620 5876 50  0000 L CNN
+F 0 "R4" H 10620 5876 50  0000 L CNN
 F 1 "470" H 10620 5784 50  0000 L CNN
 F 2 "smd:SM0603" H 10620 5708 30  0000 L CNN
@@
 $EndComp
 $Comp
-L C_Small C17
+L C_Small C8
 U 1 1 562BB6B5
 P 2250 3600
-F 0 "C17" H 2260 3670 50  0000 L CNN
+F 0 "C8" H 2260 3670 50  0000 L CNN
 F 1 "10pF" H 2260 3520 50  0000 L CNN
 F 2 "smd:SM0603" H 2250 3600 60  0001 C CNN
@@
 $EndComp
 $Comp
-L C_Small C19
+L C_Small C9
 U 1 1 562BB746
 P 2800 3600
-F 0 "C19" H 2810 3670 50  0000 L CNN
+F 0 "C9" H 2810 3670 50  0000 L CNN
 F 1 "10pF" H 2810 3520 50  0000 L CNN
 F 2 "smd:SM0603" H 2800 3600 60  0001 C CNN
@@
 RTC_OSC_OUT
 $Comp
-L CONN_01X16 P2
+L CONN_01X16 P4
 U 1 1 56324CF9
 P 7550 1750
-F 0 "P2" H 7550 2600 50  0000 C CNN
+F 0 "P4" H 7550 2600 50  0000 C CNN
 F 1 "Analog" H 7550 900 50  0000 C CNN
 F 2 "engstad:pin-strip-16" H 7550 1750 60  0001 C CNN
@@
 $EndComp
 $Comp
-L CONN_01X16 P3
+L CONN_01X16 P5
 U 1 1 5632536D
 P 8750 1750
-F 0 "P3" H 8750 2600 50  0000 C CNN
+F 0 "P5" H 8750 2600 50  0000 C CNN
 F 1 "Digital" H 8750 900 50  0000 C CNN
 F 2 "engstad:pin-strip-16" H 8750 1750 60  0001 C CNN
@@
 NoConn ~ 10800 3600
 $Comp
-L C C16
+L C C2
 U 1 1 563870A0
-P 5200 1150
-F 0 "C16" H 5225 1250 50  0000 L CNN
-F 1 "1uF" H 5225 1050 50  0000 L CNN
-F 2 "smd:SM0805" H 5238 1000 30  0001 C CNN
-F 3 "" H 5200 1150 60  0000 C CNN
-	1    5200 1150
-	1    0    0    -1
-$EndComp
-$Comp
-L C C15
+P 5200 1200
+F 0 "C2" H 5225 1300 50  0000 L CNN
+F 1 "1uF" H 5225 1100 50  0000 L CNN
+F 2 "smd:SM0805" H 5238 1050 30  0001 C CNN
+F 3 "" H 5200 1200 60  0000 C CNN
+	1    5200 1200
+	1    0    0    -1
+$EndComp
+$Comp
+L C C3
 U 1 1 564EFD30
 P 9350 1250
-F 0 "C15" H 9375 1350 50  0000 L CNN
+F 0 "C3" H 9375 1350 50  0000 L CNN
 F 1 "0.1uF" H 9375 1150 50  0000 L CNN
 F 2 "smd:SM0603" H 9388 1100 30  0001 C CNN
@@
 OTG_5V
 $Comp
-L CONN_01X02 P8
+L CONN_01X02 P6
 U 1 1 56691320
 P 4400 4050
-F 0 "P8" H 4400 4200 50  0000 C CNN
+F 0 "P6" H 4400 4200 50  0000 C CNN
 F 1 "BATT" V 4500 4050 50  0000 C CNN
 F 2 "engstad:pin-socket-2" H 4400 4050 60  0001 C CNN
@@
 $EndComp
 $Comp
-L CONN_01X01 P5
+L CONN_01X01 P1
 U 1 1 567785D7
 P 2250 650
-F 0 "P5" H 2250 550 50  0000 C CNN
+F 0 "P1" H 2250 550 50  0000 C CNN
 F 1 "VIN" H 2400 650 50  0000 C CNN
 F 2 "engstad:pin-strip-1" H 2169 510 50  0001 C CNN
@@
 VDD
 $Comp
-L spdp-2x SW2
+L spdp-2x SW1
 U 1 1 567A978A
 P 5000 3100
-F 0 "SW2" H 5000 3453 60  0000 C CNN
+F 0 "SW1" H 5000 3453 60  0000 C CNN
 F 1 "spdp-2x" H 5000 3347 60  0000 C CNN
 F 2 "engstad:slide-switch-smd-cas-220-d20" H 5000 3100 60  0001 C CNN
@@
 $EndComp
 $Comp
-L spdp-2x SW2
+L spdp-2x SW1
 U 2 1 567A9897
 P 5250 3900
-F 0 "SW2" H 5250 4150 60  0000 C CNN
+F 0 "SW1" H 5250 4150 60  0000 C CNN
 F 1 "spdp-2x" H 5250 3700 60  0000 C CNN
 F 2 "engstad:slide-switch-smd-cas-220-d20" H 5250 3900 60  0001 C CNN
@@
 $EndComp
 $Comp
-L R_Small R7
+L R_Small R1
 U 1 1 56B9F4E7
 P 1350 1900
-F 0 "R7" V 1153 1900 50  0000 C CNN
+F 0 "R1" V 1153 1900 50  0000 C CNN
 F 1 "1M0" V 1245 1900 50  0000 C CNN
 F 2 "smd:SM0603" V 1245 1900 50  0001 C CNN
@@
 $EndComp
 $Comp
-L C_Small C20
+L C_Small C4
 U 1 1 56B9F5A7
 P 1350 2100
-F 0 "C20" V 1250 2100 50  0000 C CNN
+F 0 "C4" V 1250 2100 50  0000 C CNN
 F 1 "4.7uF" V 1500 2100 50  0000 C CNN
 F 2 "smd:SM0603" H 1350 2100 50  0001 C CNN
@@
 ~MR
 $Comp
-L SW_PUSH_NO SW1
+L SW_PUSH_NO SW2
 U 1 1 567471F1
 P 9650 3500
-F 0 "SW1" H 9650 3650 60  0000 C CNN
+F 0 "SW2" H 9650 3650 60  0000 C CNN
 F 1 "RST" H 9650 3400 60  0000 C CNN
 F 2 "engstad:tactile-switch-evpay-34x29mm" H 9650 3605 60  0001 C CNN
@@
 $EndComp
 $Comp
-L CONN_01X01 P9
+L CONN_01X01 P2
 U 1 1 56DBFE79
 P 5950 950
-F 0 "P9" H 5950 850 50  0000 C CNN
+F 0 "P2" H 5950 850 50  0000 C CNN
 F 1 "VDD" H 6100 950 50  0000 C CNN
 F 2 "engstad:pin-strip-1" H 5869 810 50  0001 C CNN
@@
 $EndComp
 $Comp
-L C C12
+L C C11
 U 1 1 57D7DBA4
 P 1700 4650
-F 0 "C12" H 1500 4750 50  0000 L CNN
+F 0 "C11" H 1500 4750 50  0000 L CNN
 F 1 "0.1uF" H 1450 4550 50  0000 L CNN
 F 2 "smd:SM0603" H 1738 4500 30  0001 C CNN
@@
 $EndComp
 $Comp
-L LP5907MFX U4
+L LP5907MFX U1
 U 1 1 58FD570E
 P 4500 1050
-F 0 "U4" H 4500 1417 50  0000 C CNN
+F 0 "U1" H 4500 1417 50  0000 C CNN
 F 1 "LP5907MFX" H 4500 1326 50  0000 C CNN
 F 2 "TO_SOT_Packages_SMD:SOT-23-5" H 4500 1050 50  0001 C CNN
@@
 L GND #PWR034
 U 1 1 58FDC855
-P 5200 1300
-F 0 "#PWR034" H 5200 1050 50  0001 C CNN
-F 1 "GND" H 5200 1150 50  0000 C CNN
-F 2 "" H 5200 1300 60  0000 C CNN
-F 3 "" H 5200 1300 60  0000 C CNN
-	1    5200 1300
+P 5200 1350
+F 0 "#PWR034" H 5200 1100 50  0001 C CNN
+F 1 "GND" H 5200 1200 50  0000 C CNN
+F 2 "" H 5200 1350 60  0000 C CNN
+F 3 "" H 5200 1350 60  0000 C CNN
+	1    5200 1350
 	1    0    0    -1
 $EndComp
@@
 	4700 4100 4700 4150
 Wire Wire Line
-	5200 950  5200 1000
+	5200 950  5200 1050
 Connection ~ 5500 950
 Connection ~ 5200 950
@@
 Wire Wire Line
 	1700 1900 2050 1900
+Text Notes 9400 2800 0    45   ~ 0
+The APX823's manual reset line (~MR~) \nhas internal pullup of 60 kOhm.\n
 $EndSCHEMATC

Commit message: Working towards 0.9.
- Remove NJTRST and NRST confusion
- Remove VBUS, not needed for upstream facing port.
- Remove shielding, don't mess with the upstream ground.
- Put back SDMMC, it's not the same as QSPI.
- Add README.md.
Parts:
- removed C4: 4.7uF, smd:SM0603, symbol C_Small
- removed J1: USB_OTG, engstad:usb-micro-b-amphenol-fci-10118194, symbol USB_OTG
- removed L1, L2: Bead, smd:SM0805, symbol L_Small
- removed R1: 1M0, smd:SM0603, symbol R_Small
- removed U2: RClamp0504S, TO_SOT_Packages_SMD:SOT-23-6, symbol RClamp0504S
- removed U5: N25Q00AA, SMD_Packages:SO-16-W, symbol N25Q00AA
- added FB1, FB2: 220Ω@100MHz, Inductor_SMD:L_0805_2012Metric, symbol Device:Ferrite_Bead_Small
- added J1: USB_B_Micro, engstad:usb-micro-b-amphenol-fci-10118194, symbol Connector:USB_B_Micro
- added J2: Micro_SD_Card, engstad:Molex_PS_105162_001, symbol Connector:Micro_SD_Card_Det1
- added U2: USBLC6-2SC6, Package_TO_SOT_SMD:SOT-23-6, symbol Power_Protection:USBLC6-2SC6
- C1, C12, C2: footprint smd:SM0805 -> Capacitor_SMD:C_0805_2012Metric; symbol C -> BetsyBoard-rescue:C
- C10, C11, C14, C15, C16, C17, C3, C5, C6, C7: footprint smd:SM0603 -> Capacitor_SMD:C_0603_1608Metric; symbol C -> BetsyBoard-rescue:C
- C13: footprint smd:SM0603 -> Capacitor_SMD:C_0805_2012Metric; symbol C -> BetsyBoard-rescue:C
- C8, C9: footprint smd:SM0603 -> Capacitor_SMD:C_0603_1608Metric; symbol C_Small -> BetsyBoard-rescue:C_Small
- D1, D2: footprint w_smd_leds:Led_0603 -> LED_SMD:LED_0603_1608Metric; symbol LED-RESCUE-BetsyBoard -> BetsyBoard-rescue:LED-RESCUE-BetsyBoard
- P1: value VIN -> VDD; symbol CONN_01X01 -> BetsyBoard-rescue:CONN_01X01
- P2: value VDD -> VBUS; symbol CONN_01X01 -> BetsyBoard-rescue:CONN_01X01
- P3: symbol CONN_02X05 -> BetsyBoard-rescue:CONN_02X05
- P4, P5: symbol CONN_01X16 -> BetsyBoard-rescue:CONN_01X16
- P6: symbol CONN_01X02 -> BetsyBoard-rescue:CONN_01X02
- P7: symbol CONN_01X01 -> BetsyBoard-rescue:CONN_01X01
- R2, R3, R4: footprint smd:SM0603 -> Resistor_SMD:R_0603_1608Metric; symbol R -> BetsyBoard-rescue:R
- SW1: value spdp-2x -> DIPSW; symbol spdp-2x -> @Engstad:spdp-2x
- SW2: symbol SW_PUSH_NO -> BetsyBoard-rescue:SW_PUSH_NO
- U1: footprint TO_SOT_Packages_SMD:SOT-23-5 -> Package_TO_SOT_SMD:SOT-23-5; symbol LP5907MFX -> BetsyBoard-rescue:LP5907MFX
- U3: footprint TO_SOT_Packages_SMD:SOT-23-5 -> Package_TO_SOT_SMD:SOT-23-5; symbol APX823 -> BetsyBoard-rescue:APX823
- U4: footprint Housings_QFP:LQFP-64_10x10mm_Pitch0.5mm -> engstad:QFP-64_10x10_Pitch0.5mm; symbol STM32L486Rx-LQFP64 -> @Engstad:STM32L486Rx-LQFP64
- X1: symbol crystal-resonator-smd -> @Engstad:crystal-resonator-smd
- Y1: footprint armory:CRYSTAL-32k-B -> Crystal:Crystal_SMD_3215-2Pin_3.2x1.5mm; symbol Crystal -> BetsyBoard-rescue:Crystal
Connections:
- net labels added: D+, D-, SDMMC_DET, VBUS, ~JTRST
- net labels removed: Earth, OTG_5V, OTG_FS_ID, SHIELD, ~MR
- wire segments 108 -> 127
- no-connect marks 4 -> 5
Other:
- moved on the sheet: C1, C10, C11, C12, C13, C14, C15, C16, C17, P1, P2, P6

Commit message: More changes
Parts:
- removed U1: LP5907MFX, Package_TO_SOT_SMD:SOT-23-5, symbol BetsyBoard-rescue:LP5907MFX
- added NT1: Net-Tie_2, NetTie:NetTie-2_SMD_Pad0.5mm, symbol Device:Net-Tie_2
- added U1: LP5907MFX-3.3, Package_TO_SOT_SMD:SOT-23-5, symbol Regulator_Linear:LP5907MFX-3.3
Connections:
- net GND: now also NT1.1, U1.2 (GND); no longer U4.12 (VSSA/VREF-)
- net VDD: now also U1.5 (OUT)
- net VIN: now also U1.1 (IN), U1.3 (EN)
- new net VSSA: NT1.2, U4.12 (VSSA/VREF-)
Other:
- moved on the sheet: C6
Changed lines of the file:
@@
 L BetsyBoard-rescue:C C6
 U 1 1 55FB1A93
-P 5100 2300
-F 0 "C6" H 5125 2400 50  0000 L CNN
-F 1 "0.1uF" H 5125 2200 50  0000 L CNN
-F 2 "Capacitor_SMD:C_0603_1608Metric" H 5138 2150 30  0001 C CNN
-F 3 "" H 5100 2300 60  0000 C CNN
-	1    5100 2300
+P 5200 2300
+F 0 "C6" H 5225 2400 50  0000 L CNN
+F 1 "0.1uF" H 5225 2200 50  0000 L CNN
+F 2 "Capacitor_SMD:C_0603_1608Metric" H 5238 2150 30  0001 C CNN
+F 3 "" H 5200 2300 60  0000 C CNN
+	1    5200 2300
 	1    0    0    -1
 $EndComp
@@
 $EndComp
 $Comp
-L BetsyBoard-rescue:GND #PWR010
-U 1 1 5629DE3D
-P 5100 2450
-F 0 "#PWR010" H 5100 2200 50  0001 C CNN
-F 1 "GND" H 5100 2300 50  0000 C CNN
-F 2 "" H 5100 2450 60  0000 C CNN
-F 3 "" H 5100 2450 60  0000 C CNN
-	1    5100 2450
-	1    0    0    -1
-$EndComp
-$Comp
 L BetsyBoard-rescue:VDD #PWR011
 U 1 1 5629E0D9
@@
 	1    0    0    -1
 $EndComp
-$Comp
-L BetsyBoard-rescue:LP5907MFX U1
-U 1 1 58FD570E
-P 4500 1050
-F 0 "U1" H 4500 1417 50  0000 C CNN
-F 1 "LP5907MFX" H 4500 1326 50  0000 C CNN
-F 2 "Package_TO_SOT_SMD:SOT-23-5" H 4500 1050 50  0001 C CNN
-F 3 "" H 4500 1050 50  0000 C CNN
-	1    4500 1050
-	1    0    0    -1
-$EndComp
 Text Label 3450 950  0    60   ~ 0
 VIN
@@
 	4750 2100 4750 2150
 Wire Wire Line
-	5100 2100 5100 2150
+	5200 2100 5200 2150
 Connection ~ 4750 2100
-Connection ~ 5100 2100
+Connection ~ 5200 2100
 Wire Wire Line
 	4150 2100 3850 2100
@@
 	5900 3100 6200 3100
 Wire Wire Line
-	3900 950  3900 1150
-Wire Wire Line
-	3900 1150 4200 1150
+	3900 950  3900 1050
+Wire Wire Line
+	3900 1050 4200 1050
 Connection ~ 3900 950
 Wire Wire Line
@@
 L BetsyBoard-rescue:VDDA #PWR039
 U 1 1 58FDF596
-P 5600 2050
-F 0 "#PWR039" H 5600 1900 50  0001 C CNN
-F 1 "VDDA" H 5600 2200 50  0000 C CNN
-F 2 "" H 5600 2050 50  0001 C CNN
-F 3 "" H 5600 2050 50  0001 C CNN
-	1    5600 2050
-	1    0    0    -1
-$EndComp
-Wire Wire Line
-	5600 2100 5600 2050
+P 5850 2050
+F 0 "#PWR039" H 5850 1900 50  0001 C CNN
+F 1 "VDDA" H 5850 2200 50  0000 C CNN
+F 2 "" H 5850 2050 50  0001 C CNN
+F 3 "" H 5850 2050 50  0001 C CNN
+	1    5850 2050
+	1    0    0    -1
+$EndComp
+Wire Wire Line
+	5850 2100 5850 2050
 $Comp
 L BetsyBoard-rescue:VDDA #PWR040
@@
 L BetsyBoard-rescue:GND #PWR042
 U 1 1 58FE0727
-P 6050 6200
-F 0 "#PWR042" H 6050 5950 50  0001 C CNN
-F 1 "GND" V 6055 6072 50  0000 R CNN
-F 2 "" H 6050 6200 50  0001 C CNN
-F 3 "" H 6050 6200 50  0001 C CNN
-	1    6050 6200
-	0    1    1    0
-$EndComp
-Wire Wire Line
-	6050 6200 6100 6200
-Wire Wire Line
-	6200 5800 6100 5800
-Wire Wire Line
-	6100 5800 6100 5900
+P 6000 6200
+F 0 "#PWR042" H 6000 5950 50  0001 C CNN
+F 1 "GND" V 6005 6072 50  0000 R CNN
+F 2 "" H 6000 6200 50  0001 C CNN
+F 3 "" H 6000 6200 50  0001 C CNN
+	1    6000 6200
+	1    0    0    -1
+$EndComp
+Wire Wire Line
+	6000 6200 6100 6200
 Connection ~ 6100 6200
 Wire Wire Line
 	6200 5900 6100 5900
-Connection ~ 6100 5900
 Wire Wire Line
 	6200 6000 6100 6000
@@
 	3450 950  3650 950
 Wire Wire Line
-	4750 2100 5100 2100
-Wire Wire Line
-	5100 2100 5600 2100
+	4750 2100 5200 2100
+Wire Wire Line
+	5200 2100 5850 2100
 Wire Wire Line
 	2250 3400 2400 3400
@@
 Wire Wire Line
 	5500 3900 5500 4000
+$Comp
+L Regulator_Linear:LP5907MFX-3.3 U1
+U 1 1 5F6ED042
+P 4500 1050
+F 0 "U1" H 4500 1417 50  0000 C CNN
+F 1 "LP5907MFX-3.3" H 4500 1326 50  0000 C CNN
+F 2 "Package_TO_SOT_SMD:SOT-23-5" H 4500 1400 50  0001 C CNN
+F 3 "http://www.ti.com/lit/ds/symlink/lp5907.pdf" H 4500 1550 50  0001 C CNN
+	1    4500 1050
+	1    0    0    -1
+$EndComp
+$Comp
+L power:VSSA #PWR0103
+U 1 1 5F7AACB0
+P 6000 5800
+F 0 "#PWR0103" H 6000 5650 50  0001 C CNN
+F 1 "VSSA" H 6015 5973 50  0000 C CNN
+F 2 "" H 6000 5800 50  0001 C CNN
+F 3 "" H 6000 5800 50  0001 C CNN
+	1    6000 5800
+	-1   0    0    1
+$EndComp
+Wire Wire Line
+	6000 5800 6200 5800
+$Comp
+L Device:Net-Tie_2 NT1
+U 1 1 5F7C24DA
+P 5750 2450
+F 0 "NT1" H 5750 2631 50  0000 C CNN
+F 1 "Net-Tie_2" H 5750 2540 50  0000 C CNN
+F 2 "NetTie:NetTie-2_SMD_Pad0.5mm" H 5750 2450 50  0001 C CNN
+F 3 "~" H 5750 2450 50  0001 C CNN
+	1    5750 2450
+	1    0    0    -1
+$EndComp
+$Comp
+L BetsyBoard-rescue:GND #PWR0104
+U 1 1 5F7D17B7
+P 5650 2450
+F 0 "#PWR0104" H 5650 2200 50  0001 C CNN
+F 1 "GND" H 5650 2300 50  0000 C CNN
+F 2 "" H 5650 2450 60  0000 C CNN
+F 3 "" H 5650 2450 60  0000 C CNN
+	1    5650 2450
+	1    0    0    -1
+$EndComp
+$Comp
+L power:VSSA #PWR0105
+U 1 1 5F7D22B3
+P 5850 2450
+F 0 "#PWR0105" H 5850 2300 50  0001 C CNN
+F 1 "VSSA" H 5850 2600 50  0000 C CNN
+F 2 "" H 5850 2450 50  0001 C CNN
+F 3 "" H 5850 2450 50  0001 C CNN
+	1    5850 2450
+	-1   0    0    1
+$EndComp
+$Comp
+L BetsyBoard-rescue:GND #PWR?
+U 1 1 5F817E0A
+P 5200 2450
+F 0 "#PWR?" H 5200 2200 50  0001 C CNN
+F 1 "GND" H 5200 2300 50  0000 C CNN
+F 2 "" H 5200 2450 60  0000 C CNN
+F 3 "" H 5200 2450 60  0000 C CNN
+	1    5200 2450
+	1    0    0    -1
+$EndComp
 $EndSCHEMATC

Commit message: Fix rescued symbols
Parts:
- C1, C10, C11, C12, C13, C14, C15, C16, C17, C2, C3, C5, C6, C7: symbol BetsyBoard-rescue:C -> Device:C
- C8, C9: symbol BetsyBoard-rescue:C_Small -> Device:C_Small
- D1, D2: symbol BetsyBoard-rescue:LED-RESCUE-BetsyBoard -> Device:LED
- P1, P2: symbol BetsyBoard-rescue:CONN_01X01 -> Connector:Conn_01x01_Male
- P3: symbol BetsyBoard-rescue:CONN_02X05 -> Connector_Generic:Conn_02x05_Odd_Even
- P4, P5: symbol BetsyBoard-rescue:CONN_01X16 -> Connector_Generic:Conn_01x16
- P6: symbol BetsyBoard-rescue:CONN_01X02 -> Connector_Generic:Conn_01x02
- P7: symbol BetsyBoard-rescue:CONN_01X01 -> Connector_Generic:Conn_01x01
- R2, R3, R4: symbol BetsyBoard-rescue:R -> Device:R
- SW2: symbol BetsyBoard-rescue:SW_PUSH_NO -> @Engstad:SW_PUSH_NO
- U3: symbol BetsyBoard-rescue:APX823 -> @Engstad:APX823
- Y1: symbol BetsyBoard-rescue:Crystal -> Device:Crystal

Commit message: Major changes due to mistakes
Parts:
- J1: footprint engstad:usb-micro-b-amphenol-fci-10118194 -> engstad:usb-micro-b-amphenol-fci-10118194-oval
- P3: Manu# (none) -> FTSH-105-01-F-DV-K-A; Mouser# (none) -> 200-FTSH10501LDV007K
Connections:
- net labels added: LED, RESET#
- net labels removed: ~JTRST
- wire segments 126 -> 128
- no-connect marks 5 -> 6
Changed lines of the file:
@@
 Text Label 9100 4600 0    60   ~ 0
 JTDI
-Text Label 9100 4900 0    60   ~ 0
+Text Label 9100 5700 0    60   ~ 0
 D1
-Text Label 9100 5700 0    60   ~ 0
+Text Label 9100 5800 0    60   ~ 0
 D2
-Text Label 9100 5800 0    60   ~ 0
+Text Label 9100 5900 0    60   ~ 0
 D3
-Text Label 9100 6000 0    60   ~ 0
+Text Label 9100 6100 0    60   ~ 0
 D5
-Text Label 9100 6100 0    60   ~ 0
+Text Label 9100 6200 0    60   ~ 0
 D6
-Text Label 9100 6200 0    60   ~ 0
+Text Label 6200 4500 2    60   ~ 0
 D7
-Text Label 6200 4500 2    60   ~ 0
+Text Label 6200 4600 2    60   ~ 0
 D8
-Text Label 6200 4600 2    60   ~ 0
+Text Label 9100 4000 0    60   ~ 0
 D9
 Text Label 9100 5200 0    60   ~ 0
@@
 Text Label 6200 3300 2    60   ~ 0
 RTC
-Text Label 9100 5900 0    60   ~ 0
+Text Label 9100 6000 0    60   ~ 0
 D4
 Text Label 10300 1350 0    60   ~ 0
@@
 F 2 "engstad:conn-jtag-0.05" H 10000 50  60  0001 C CNN
 F 3 "" H 10000 50  60  0000 C CNN
+F 4 "200-FTSH10501LDV007K" H 10000 1250 50  0001 C CNN "Mouser#"
+F 5 "FTSH-105-01-F-DV-K-A" H 10000 1250 50  0001 C CNN "Manu#"
 	1    10000 1250
 	1    0    0    -1
 $EndComp
-Text Label 9100 4000 0    60   ~ 0
+Text Label 9100 4100 0    60   ~ 0
 D10
-Text Label 9100 4100 0    60   ~ 0
+Text Label 9100 5100 0    60   ~ 0
 D11
 Text Label 9100 5300 0    60   ~ 0
@@
 	1    0    0    -1
 $EndComp
-Text Label 10150 4950 0    60   ~ 0
-D1
 $Comp
 L power:GND #PWR05
@@
 Text Label 5600 3100 2    60   ~ 0
 BOOT_SEL
-Text Label 10300 1450 0    60   ~ 0
-~JTRST
 $Comp
 L @Engstad:SW_PUSH_NO SW2
@@
 F 0 "J1" H 1257 1617 50  0000 C CNN
 F 1 "USB_B_Micro" H 1257 1526 50  0000 C CNN
-F 2 "engstad:usb-micro-b-amphenol-fci-10118194" H 1350 1100 50  0001 C CNN
+F 2 "engstad:usb-micro-b-amphenol-fci-10118194-oval" H 1350 1100 50  0001 C CNN
 F 3 "~" H 1350 1100 50  0001 C CNN
 	1    1200 1150
@@
 Text Label 2000 950  0    50   ~ 0
 VBUS
-Text Label 9100 5100 0    60   ~ 0
-~JTRST
 Wire Wire Line
 	9800 3500 9900 3500
@@
 $EndComp
 $Comp
-L power:GND #PWR?
+L power:GND #PWR0106
 U 1 1 5F817E0A
 P 5200 2450
-F 0 "#PWR?" H 5200 2200 50  0001 C CNN
+F 0 "#PWR0106" H 5200 2200 50  0001 C CNN
 F 1 "GND" H 5200 2300 50  0000 C CNN
 F 2 "" H 5200 2450 60  0000 C CNN
@@
 	2450 650  2750 650
 $Comp
-L power:PWR_FLAG #FLG?
+L power:PWR_FLAG #FLG0101
 U 1 1 5F72B5EE
 P 3650 800
-F 0 "#FLG?" H 3650 875 50  0001 C CNN
+F 0 "#FLG0101" H 3650 875 50  0001 C CNN
 F 1 "PWR_FLAG" H 3650 973 50  0000 C CNN
 F 2 "" H 3650 800 50  0001 C CNN
@@
 	1    0    0    -1
 $EndComp
+Text Label 10300 1450 0    50   ~ 0
+RESET#
+Text Label 9700 3200 2    50   ~ 0
+RESET#
+Wire Wire Line
+	9700 3200 9800 3200
+Wire Wire Line
+	9800 3200 9800 3500
+Connection ~ 9800 3500
+NoConn ~ 5100 4800
+Text Label 9100 4900 0    60   ~ 0
+LED
+Text Label 10150 4950 0    60   ~ 0
+LED
 $EndSCHEMATC

Commit message: Version 0.9c of BetsyBoard
Parts:
- removed FB1: 220Ω@100MHz, Inductor_SMD:L_0805_2012Metric, symbol Device:Ferrite_Bead_Small
- removed P6: BATT, engstad:pin-socket-2, symbol Connector_Generic:Conn_01x02
- removed SW1: DIPSW, engstad:slide-switch-smd-cas-220-d20, symbol @Engstad:spdp-2x
- added C18, C4: 10pF, Capacitor_SMD:C_0603_1608Metric, symbol Device:C_Small
- added F1: Fuse_Small, Fuse:Fuse_0805_2012Metric, symbol Device:Fuse_Small
- added P6: VDD, Connector_PinHeader_2.54mm:PinHeader_1x01_P2.54mm_Vertical, symbol Connector:Conn_01x01_Male
- J1: symbol Connector:USB_B_Micro -> BetsyBoard-rescue:USB_B_Micro-Connector
- J2: symbol Connector:Micro_SD_Card_Det1 -> BetsyBoard-rescue:Micro_SD_Card_Det1-Connector
- NT1: footprint NetTie:NetTie-2_SMD_Pad0.5mm -> engstad:net-tie-0.4mm
- P7: value RTC -> MCO
- U4: symbol @Engstad:STM32L486Rx-LQFP64 -> BetsyBoard-rescue:STM32L486Rx-LQFP64-@Engstad
Connections:
- net labels added: MCO
- net labels removed: RTC, VBAT_IN
- no-connect marks 6 -> 4
Other:
- moved on the sheet: C8, C9, Y1
