File: BetsyBoardBig.sch (KiCad schematic (older format))
At the start: 42 parts, among them J1 USB_B_Micro, J2 Micro_SD_Card, P1 VDD, P2 VBUS, P3 CORTEX-JTAG, P4 Analog, P5 Digital, P6 BATT, P7 RTC, SW1 DIPSW, SW2 RST, U1 LP5907MFX-3.3, U2 USBLC6-2SC6, U3 APX823, U4 STM32L486Rx-LQFP64, U5 IS25WP256D-xM, X1 XTAL, Y1 Crystal

Commit message: Changes to the BBB.
- Fixing the QSPI_SCK problem.
- Cleaning up.
Parts:
- removed C13: 1.0uF, Capacitor_SMD:C_0805_2012Metric, symbol Device:C
- removed P1: VDD, engstad:pin-strip-1, symbol Connector:Conn_01x01_Male
- removed P2: VBUS, engstad:pin-strip-1, symbol Connector:Conn_01x01_Male
- removed P4: Analog, engstad:pin-strip-16, symbol Connector_Generic:Conn_01x16
- removed P5: Digital, engstad:pin-strip-16, symbol Connector_Generic:Conn_01x16
- removed P7: RTC, engstad:pin-socket-1, symbol Connector_Generic:Conn_01x01
- added C13, C18: 10pF, Capacitor_SMD:C_0603_1608Metric, symbol Device:C_Small
- added C4: 0.1uF, Capacitor_SMD:C_0603_1608Metric, symbol Device:C
- added H1, H2, H3, H4: Mounting, MountingHole:MountingHole_3.2mm_M3_Pad_Via, symbol Mechanical:MountingHole_Pad
- added J3: CLOCKS, Connector_PinHeader_2.54mm:PinHeader_2x05_P2.54mm_Vertical, symbol Connector_Generic:Conn_02x05_Odd_Even
- added J4: USART3, Connector_PinHeader_2.54mm:PinHeader_1x08_P2.54mm_Horizontal, symbol Connector_Generic:Conn_01x08
- added J5: SPI/USART, Connector_PinSocket_2.54mm:PinSocket_2x05_P2.54mm_Vertical, symbol Connector_Generic:Conn_02x05_Odd_Even
- added J6: I2C, Connector_JST:JST_SH_SM04B-SRSS-TB_1x04-1MP_P1.00mm_Horizontal, symbol Connector_Generic:Conn_01x04
- added J7: ANALOG, Connector_PinHeader_2.54mm:PinHeader_1x10_P2.54mm_Horizontal, symbol Connector_Generic:Conn_01x10
- added R1: 1K, Resistor_SMD:R_0603_1608Metric, symbol Device:R
- added R5, R6, R7: 10K, Resistor_SMD:R_0603_1608Metric, symbol Device:R
- added SW3: USR, engstad:tactile-switch-evpay-34x29mm, symbol @Engstad:SW_PUSH_NO
- added U6: 74LVC1G3157, Package_TO_SOT_SMD:SOT-23-6, symbol 74xGxx:74LVC1G3157
- D2: value GREEN -> GRN
- J1: footprint engstad:usb-micro-b-amphenol-fci-10118194 -> engstad:usb-micro-b-amphenol-fci-10118194-oval
- U4: footprint engstad:QFP-64_10x10_Pitch0.5mm -> Package_QFP:LQFP-64_10x10mm_P0.5mm
Connections:
- net labels added: BTN, COMP_IN+, COMP_IN-, COMP_OUT, DAC_OUT1, DAC_OUT2, I2C_SCL, I2C_SDA, LED_RED, OCLK_LS, OCLK_M, OPAMP_IN+, OPAMP_IN-, OPAMP_OUT, PB13, RTC_OUT, RTC_REFIN, RTC_TS, SEL_USART3, SPI2_MISO, SPI2_MOSI, SPI2_SCK, SPI2_SS#, SWCLK, SWDIO, SWO, USART1_RX, USART1_TX, USART3_CK, USART3_CTS, USART3_RTS, USART3_RXD, USART3_TXD, USR, USR_SW
- net labels removed: A1, A10, A11, A12, A2, A3, A4, A5, A6, A7, A8, A9, D1, D10, D11, D12, D13, D14, D15, D16, D2, D3, D4, D5, D6, D7, D8, D9, JTCK/SWCLK, JTDI, JTDO/SWO, JTMS/SWDIO, RTC, ~JTRST
- wire segments 125 -> 151
- no-connect marks 5 -> 7
Other:
- note added: "Changes from v0.1:\n- Pin 29 connected to SPI2_SCK changed to QSPI_SCK (and hooked up).\n- Pin 34 connected to USART3_CTS changed to PB13.\n- Removed JTAG support (pin 50 (PA15) and 56 (PB4)), now only support SWD.\n- SDMMC_DET (pin 38 (PC7)) moved to pin 50 (PA15).\n- LED_RED (pin 61 (PB8)) moved to pin 38 (PC7).\n- Removed VBUS and VCC test-points.\n- Added 74LVC1G157 connecting SEL_USART3 (pin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"
- note added: "SEL_USART3 = 0 : SPI2_SCK <- PB13\nSEL_USART3 = 1 : USART3_CTS -> PB13"
- note added: "USART1_CK: PA8, PB5 \nUSART1_TX: PA9, PB6\nUSART1_RX: PA10, PB7\nUSART1_CTS: PA11, PB4\nUSART1_RTS_DE: PA12, PB3"
- note added: "USART2_CTS: PA0\nUSART2_RTS: PA1\nUSART2_TX: PA2\nUSART2_RX: PA3\nUSART2_CK: PA4"
- note added: "USART3_CTS: PA6, PB13\nUSART3_RTS: PB1, PB14, PD2\nUSART3_TX: PC4, PB10, PC10\nUSART3_RX: PC5, PB11, PC11\nUSART3_CK: PB0, PB12, PC12"
- moved on the sheet: C10, C11, C12, C14, C15, C16, C17, C3, C5, C6, C7, C8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

Commit message: Major changes due to mistakes
Parts:
- removed SW1: DIPSW, engstad:slide-switch-smd-cas-220-d20, symbol @Engstad:spdp-2x
- added SW1: JUMPER_x2, Connector_PinHeader_2.54mm:PinHeader_2x03_P2.54mm_Vertical, symbol @Engstad:JUMPER_x2
- J2: DigiKey# (none) -> WM14405CT-ND
- J5: footprint Connector_PinSocket_2.54mm:PinSocket_2x05_P2.54mm_Vertical -> Connector_PinHeader_2.54mm:PinHeader_2x05_P2.54mm_Vertical
- SW3: DigiKey# (none) -> ‎P17064CT-ND‎; Manuf# (none) -> ‎EVP-AYF1BA‎
- U1: value LP5907MFX-3.3 -> TLV75733PDBVR‎
- U3: DigKey# (none) -> APX823-31W5GDICT-ND
Connections:
- net labels added: JTDI, RSTIN#, SWCLK_JTCK, SWDIO_JTMS, SWO_JTDO, USR_BTN
- net labels removed: BTN, RTC_REFIN, SWCLK, SWDIO, SWO, USR
- wire segments 151 -> 155
- no-connect marks 7 -> 6
Other:
- note added: "Changes from v0.1:\n- Pin 29 connected to SPI2_SCK changed to QSPI_SCK (and hooked up).\n- Pin 34 connected to USART3_CTS changed to PB13.\n- Removed NJTRST pin PB4.\n- SDMMC_DET (pin 38 (PC7)) moved to pin 56 (PB4).\n- LED_RED (pin 61 (PB8)) moved to pin 38 (PC7).\n- Removed VBUS and VCC test-points.\n- Added 74LVC1G157 connecting SEL_USART3 (pin 36 (PB15)) and PB13 (pin 34) <-> USART3_CTS and S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"
- note added: "Flipped direction of all these pins \n(except USART), double check!"
- note added: "Pin 7 was connected to PB15."
- note removed: "Changes from v0.1:\n- Pin 29 connected to SPI2_SCK changed to QSPI_SCK (and hooked up).\n- Pin 34 connected to USART3_CTS changed to PB13.\n- Removed JTAG support (pin 50 (PA15) and 56 (PB4)), now only support SWD.\n- SDMMC_DET (pin 38 (PC7)) moved to pin 50 (PA15).\n- LED_RED (pin 61 (PB8)) moved to pin 38 (PC7).\n- Removed VBUS and VCC test-points.\n- Added 74LVC1G157 connecting SEL_USART3 (pin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"
- moved on the sheet: SW2
Changed lines of the file:
@@
 OTG_FS_D+
 Text Label 10550 4500 0    50   ~ 0
-SWDIO
+SWDIO_JTMS
 $Comp
 L Device:C C12
@@
 SDMMC_D2
 Text Label 10550 4600 0    50   ~ 0
-SWCLK
+SWCLK_JTCK
 Text Label 7650 3400 2    50   ~ 0
 RTC_TS
-Text Label 10650 1000 0    60   ~ 0
-SWO
+Text Label 10650 1000 0    50   ~ 0
+SWO_JTDO
 $Comp
 L Device:C C10
@@
 	1    0    0    -1
 $EndComp
-Text Label 10650 800  0    60   ~ 0
-SWDIO
-Text Label 10650 900  0    60   ~ 0
-SWCLK
+Text Label 10650 800  0    50   ~ 0
+SWDIO_JTMS
+Text Label 10650 900  0    50   ~ 0
+SWCLK_JTCK
 $Comp
 L Device:LED D1
@@
 L power:GND #PWR024
 U 1 1 5674E8E6
-P 5050 5000
-F 0 "#PWR024" H 5050 4750 50  0001 C CNN
-F 1 "GND" H 5050 4850 50  0000 C CNN
-F 2 "" H 5050 5000 60  0000 C CNN
-F 3 "" H 5050 5000 60  0000 C CNN
-	1    5050 5000
-	1    0    0    -1
-$EndComp
-$Comp
-L @Engstad:spdp-2x SW1
-U 1 1 567A978A
-P 4200 3950
-F 0 "SW1" H 4200 4200 60  0000 C CNN
-F 1 "DIPSW" H 4200 3700 60  0000 C CNN
-F 2 "engstad:slide-switch-smd-cas-220-d20" H 4200 3950 60  0001 C CNN
-F 3 "" H 4200 3950 60  0000 C CNN
-	1    4200 3950
-	-1   0    0    1
-$EndComp
-$Comp
-L @Engstad:spdp-2x SW1
-U 2 1 567A9897
-P 3850 3150
-F 0 "SW1" H 3850 2900 60  0000 C CNN
-F 1 "DIPSW" H 3850 3400 60  0000 C CNN
-F 2 "engstad:slide-switch-smd-cas-220-d20" H 3850 3150 60  0001 C CNN
-F 3 "" H 3850 3150 60  0000 C CNN
-	2    3850 3150
-	-1   0    0    -1
+P 4950 5000
+F 0 "#PWR024" H 4950 4750 50  0001 C CNN
+F 1 "GND" H 4950 4850 50  0000 C CNN
+F 2 "" H 4950 5000 60  0000 C CNN
+F 3 "" H 4950 5000 60  0000 C CNN
+	1    4950 5000
+	1    0    0    -1
 $EndComp
 Text Label 7650 3300 2    50   ~ 0
@@
 L @Engstad:SW_PUSH_NO SW2
 U 1 1 567471F1
-P 5200 4900
-F 0 "SW2" H 5200 5050 60  0000 C CNN
-F 1 "RST" H 5200 4800 60  0000 C CNN
-F 2 "engstad:tactile-switch-evpay-34x29mm" H 5200 5005 60  0001 C CNN
-F 3 "" H 5200 4900 60  0000 C CNN
-	1    5200 4900
+P 5100 4900
+F 0 "SW2" H 5100 5050 60  0000 C CNN
+F 1 "RST" H 5100 4800 60  0000 C CNN
+F 2 "engstad:tactile-switch-evpay-34x29mm" H 5100 5005 60  0001 C CNN
+F 3 "" H 5100 4900 60  0000 C CNN
+	1    5100 4900
 	1    0    0    -1
 $EndComp
@@
 F 2 "engstad:Molex_PS_105162_001" H 3900 5600 50  0001 C CNN
 F 3 "https://www.molex.com/pdm_docs/sd/1051620001_sd.pdf" H 2750 5300 50  0001 C CNN
+F 4 "WM14405CT-ND" H 2750 5300 50  0001 C CNN "DigiKey#"
 	1    2750 5300
 	1    0    0    -1
@@
 Text Label 2750 1750 0    60   ~ 0
 OTG_FS_D-
-Text Label 10550 4700 0    50   ~ 0
+Text Label 10550 5200 0    50   ~ 0
 SDMMC_DET
 Text Label 1850 5800 2    60   ~ 0
 SDMMC_DET
 Text Label 10550 5100 0    50   ~ 0
-SWO
-Wire Wire Line
-	3600 3050 3400 3050
-Wire Wire Line
-	3600 3250 3400 3250
-Wire Wire Line
-	4100 3150 4450 3150
-Wire Wire Line
-	3400 3850 3950 3850
-Wire Wire Line
-	3650 4050 3950 4050
-Wire Wire Line
-	4450 3950 4600 3950
+SWO_JTDO
 Connection ~ 4600 3950
 Wire Wire Line
@@
 P 4500 1050
 F 0 "U1" H 4500 1417 50  0000 C CNN
-F 1 "LP5907MFX-3.3" H 4500 1326 50  0000 C CNN
+F 1 "TLV75733PDBVR‎" H 4500 1326 50  0000 C CNN
 F 2 "Package_TO_SOT_SMD:SOT-23-5" H 4500 1400 50  0001 C CNN
-F 3 "http://www.ti.com/lit/ds/symlink/lp5907.pdf" H 4500 1550 50  0001 C CNN
+F 3 "https://www.ti.com/lit/ds/symlink/tlv757p.pdf?HQS=TI-null-null-digikeymode-df-pf-null-wwe&ts=1601868242728" H 4500 1550 50  0001 C CNN
 	1    4500 1050
 	1    0    0    -1
@@
 F 2 "Package_TO_SOT_SMD:SOT-23-5" H 5800 4900 60  0001 C CNN
 F 3 "http://www.diodes.com/_files/datasheets/APX823_824_825A.pdf" V 6600 4900 60  0001 C CNN
+F 4 "APX823-31W5GDICT-ND" H 5800 4900 50  0001 C CNN "DigKey#"
 	1    5800 4900
 	1    0    0    -1
@@
 Text Label 10550 5000 0    50   ~ 0
 RTC_OUT
-Text Label 10550 6300 0    50   ~ 0
-RTC_REFIN
 Text Label 10550 4100 0    50   ~ 0
 USART1_TX
@@
 F 0 "J5" H 8350 1417 50  0000 C CNN
 F 1 "SPI/USART" H 8350 1326 50  0000 C CNN
-F 2 "Connector_PinSocket_2.54mm:PinSocket_2x05_P2.54mm_Vertical" H 8300 1000 50  0001 C CNN
+F 2 "Connector_PinHeader_2.54mm:PinHeader_2x05_P2.54mm_Vertical" H 8300 1000 50  0001 C CNN
 F 3 "~" H 8300 1000 50  0001 C CNN
 	1    8300 1000
 	1    0    0    -1
 $EndComp
+Text Label 8100 1200 2    50   ~ 0
+USART1_TX
 Text Label 8600 1200 0    50   ~ 0
-USART1_TX
-Text Label 8100 1200 2    50   ~ 0
 USART1_RX
 Text Label 8100 900  2    50   ~ 0
@@
 Text Label 6400 1000 2    50   ~ 0
 RTC_TS
-Text Label 6400 1100 2    50   ~ 0
-RTC_REFIN
 $Comp
 L power:GND #PWR036
@@
 F 2 "engstad:tactile-switch-evpay-34x29mm" H 5650 3705 60  0001 C CNN
 F 3 "" H 5650 3600 60  0000 C CNN
+F 4 "‎P17064CT-ND‎" H 5650 3600 50  0001 C CNN "DigiKey#"
+F 5 "‎EVP-AYF1BA‎" H 5650 3600 50  0001 C CNN "Manuf#"
 	1    5650 3600
 	0    -1   -1   0
@@
 OPAMP_OUT
 Wire Wire Line
-	5050 4900 5050 5000
+	4950 4900 4950 5000
 Text Label 10300 2250 2    50   ~ 0
 COMP_IN+
@@
 	2000 3050 2350 3050
 Text Label 6400 1200 2    50   ~ 0
-SWCLK
+SWCLK_JTCK
 Text Label 8100 1100 2    50   ~ 0
-SWDIO
+SWDIO_JTMS
 Text Label 8600 1100 0    50   ~ 0
-SWO
+SWO_JTDO
 Wire Wire Line
 	6400 800  6300 800
@@
 Text Label 2750 6900 2    50   ~ 0
 PB13
-NoConn ~ 10650 1100
-NoConn ~ 10650 1200
 Text Label 2750 7100 2    50   ~ 0
 SEL_USART3
-Text Label 10550 5200 0    50   ~ 0
-SEL_USART3
 Text Label 10550 5600 0    50   ~ 0
-USR
+USR_BTN
 $Comp
 L power:GND #PWR0112
@@
 	6300 2400 6850 2400
 Text Label 5650 3400 2    50   ~ 0
-BTN
+USR_BTN
 Text Notes 7000 7100 0    40   ~ 0
-Changes from v0.1:\n- Pin 29 connected to SPI2_SCK changed to QSPI_SCK (and hooked up).\n- Pin 34 connected to USART3_CTS changed to PB13.\n- Removed JTAG support (pin 50 (PA15) and 56 (PB4)), now only support SWD.\n- SDMMC_DET (pin 38 (PC7)) moved to pin 50 (PA15).\n- LED_RED (pin 61 (PB8)) moved to pin 38 (PC7).\n- Removed VBUS and VCC test-points.\n- Added 74LVC1G157 connecting SEL_USART3 (pin 56 (PB4)) and PB13 (pin 34) <-> USART3_CTS and SPI2_SCK.
+Changes from v0.1:\n- Pin 29 connected to SPI2_SCK changed to QSPI_SCK (and hooked up).\n- Pin 34 connected to USART3_CTS changed to PB13.\n- Removed NJTRST pin PB4.\n- SDMMC_DET (pin 38 (PC7)) moved to pin 56 (PB4).\n- LED_RED (pin 61 (PB8)) moved to pin 38 (PC7).\n- Removed VBUS and VCC test-points.\n- Added 74LVC1G157 connecting SEL_USART3 (pin 36 (PB15)) and PB13 (pin 34) <-> USART3_CTS and SPI2_SCK.
 Text Label 4800 3150 0    50   ~ 0
 BOOT0
@@
 	5200 3550 500  3550
 $Comp
-L power:VDD #PWR?
+L power:VDD #PWR0116
 U 1 1 5FA77FB1
 P 4550 4950
-F 0 "#PWR?" H 4550 4800 50  0001 C CNN
+F 0 "#PWR0116" H 4550 4800 50  0001 C CNN
 F 1 "VDD" H 4550 5100 50  0000 C CNN
 F 2 "" H 4550 4950 60  0000 C CNN
@@
 $EndComp
 $Comp
-L power:VDD #PWR?
+L power:VDD #PWR0117
 U 1 1 5FAACB03
 P 6650 4800
-F 0 "#PWR?" H 6650 4650 50  0001 C CNN
+F 0 "#PWR0117" H 6650 4650 50  0001 C CNN
 F 1 "VDD" H 6650 4950 50  0000 C CNN
 F 2 "" H 6650 4800 60  0000 C CNN
@@
 Wire Wire Line
 	9050 1000 9050 1200
+$Comp
+L @Engstad:JUMPER_x2 SW1
+U 1 1 5F811252
+P 3850 3150
+F 0 "SW1" H 3850 3400 60  0000 C CNN
+F 1 "JUMPER_x2" H 3850 2900 60  0000 C CNN
+F 2 "Connector_PinHeader_2.54mm:PinHeader_2x03_P2.54mm_Vertical" H 3850 3150 60  0001 C CNN
+F 3 "" H 3850 3150 60  0000 C CNN
+	1    3850 3150
+	-1   0    0    -1
+$EndComp
+Wire Wire Line
+	4000 3150 4450 3150
+Wire Wire Line
+	3400 3050 3700 3050
+Wire Wire Line
+	3400 3250 3700 3250
+$Comp
+L @Engstad:JUMPER_x2 SW1
+U 2 1 5F827D4F
+P 4200 3950
+F 0 "SW1" H 4200 4200 60  0000 C CNN
+F 1 "JUMPER_x2" H 4200 3750 60  0000 C CNN
+F 2 "Connector_PinHeader_2.54mm:PinHeader_2x03_P2.54mm_Vertical" H 4200 3950 60  0001 C CNN
+F 3 "" H 4200 3950 60  0000 C CNN
+	2    4200 3950
+	-1   0    0    -1
+$EndComp
+Wire Wire Line
+	3400 3850 4050 3850
+Wire Wire Line
+	3650 4050 4050 4050
+Wire Wire Line
+	4350 3950 4600 3950
+Wire Wire Line
+	5250 4900 5300 4900
+Wire Wire Line
+	5300 4900 5300 4650
+Wire Wire Line
+	5300 4650 5200 4650
+Connection ~ 5300 4900
+Wire Wire Line
+	5300 4900 5350 4900
+Text Label 5200 4650 2    50   ~ 0
+RSTIN#
+Text Label 10650 1200 0    50   ~ 0
+RSTIN#
+Text Notes 5850 1350 0    40   ~ 0
+Pin 7 was connected to PB15.
+NoConn ~ 6400 1100
+Text Label 10550 4700 0    50   ~ 0
+JTDI
+Text Label 10650 1100 0    50   ~ 0
+JTDI
+Text Label 10550 6300 0    50   ~ 0
+SEL_USART3
+Text Notes 7800 1400 0    40   ~ 0
+Flipped direction of all these pins \n(except USART), double check!
 $EndSCHEMATC

Commit message: More changes.
Parts:
- C13, C18: value 10pF -> 16pF
- C8, C9: value 10pF -> 12pF
- R3, R4: value 470 -> 180
Other:
- note added: "3.3V/20mA = 165 ohm (1%)\n160 (5%) or 180 (10%)"
Changed lines of the file:
@@
 P 4100 5700
 F 0 "R3" H 4030 5776 50  0000 R CNN
-F 1 "470" H 4030 5684 50  0000 R CNN
+F 1 "180" H 4030 5684 50  0000 R CNN
 F 2 "Resistor_SMD:R_0603_1608Metric" H 4030 5608 30  0001 R CNN
 F 3 "" H 4100 5700 30  0000 C CNN
@@
 P 4550 5700
 F 0 "R4" H 4620 5776 50  0000 L CNN
-F 1 "470" H 4620 5684 50  0000 L CNN
+F 1 "180" H 4620 5684 50  0000 L CNN
 F 2 "Resistor_SMD:R_0603_1608Metric" H 4620 5608 30  0001 L CNN
 F 3 "" H 4550 5700 30  0000 C CNN
@@
 P 1350 4150
 F 0 "C8" H 1360 4220 50  0000 L CNN
-F 1 "10pF" H 1360 4070 50  0000 L CNN
+F 1 "12pF" H 1360 4070 50  0000 L CNN
 F 2 "Capacitor_SMD:C_0603_1608Metric" H 1350 4150 60  0001 C CNN
 F 3 "" H 1350 4150 60  0000 C CNN
@@
 P 1900 4150
 F 0 "C9" H 1910 4220 50  0000 L CNN
-F 1 "10pF" H 1910 4070 50  0000 L CNN
+F 1 "12pF" H 1910 4070 50  0000 L CNN
 F 2 "Capacitor_SMD:C_0603_1608Metric" H 1900 4150 60  0001 C CNN
 F 3 "" H 1900 4150 60  0000 C CNN
@@
 P 1300 3200
 F 0 "C13" H 1310 3270 50  0000 L CNN
-F 1 "10pF" H 1310 3120 50  0000 L CNN
+F 1 "16pF" H 1310 3120 50  0000 L CNN
 F 2 "Capacitor_SMD:C_0603_1608Metric" H 1300 3200 60  0001 C CNN
 F 3 "" H 1300 3200 60  0000 C CNN
@@
 P 2000 3200
 F 0 "C18" H 2010 3270 50  0000 L CNN
-F 1 "10pF" H 2010 3120 50  0000 L CNN
+F 1 "16pF" H 2010 3120 50  0000 L CNN
 F 2 "Capacitor_SMD:C_0603_1608Metric" H 2000 3200 60  0001 C CNN
 F 3 "" H 2000 3200 60  0000 C CNN
@@
 Text Notes 7800 1400 0    40   ~ 0
 Flipped direction of all these pins \n(except USART), double check!
+Text Notes 3900 4750 0    40   ~ 0
+3.3V/20mA = 165 ohm (1%)\n160 (5%) or 180 (10%)
 $EndSCHEMATC

Commit message: Adding +5V support for I2C port, and fixing courtyard layer.
Parts:
- removed R6, R7: 10K, Resistor_SMD:R_0603_1608Metric, symbol Device:R
- added C19: 0.1uF, Capacitor_SMD:C_0603_1608Metric, symbol Device:C_Small
- added Q1: BSS138BKS, Package_TO_SOT_SMD:SOT-363_SC-70-6, symbol @Engstad:BSS138BKS
- added RN1: 10K, Resistor_SMD:R_Array_Concave_4x0603, symbol Device:R_Pack04_Split
- C5: footprint Capacitor_SMD:C_0603_1608Metric -> Capacitor_SMD:C_0805_2012Metric
Connections:
- net labels added: +5V, EXTSCL, EXTSDA
- wire segments 155 -> 163

Commit message: Use a battery header I can actually procure.
Parts:
- P6: footprint Connector_JST:JST_SH_BM02B-SRSS-TB_1x02-1MP_P1.00mm_Vertical -> Connector_JST:JST_PH_B2B-PH-K_1x02_P2.00mm_Vertical
Changed lines of the file:
@@
 F 0 "P6" H 3450 4150 50  0000 C CNN
 F 1 "BATT" V 3550 4000 50  0000 C CNN
-F 2 "Connector_JST:JST_SH_BM02B-SRSS-TB_1x02-1MP_P1.00mm_Vertical" H 3450 4050 60  0001 C CNN
-F 3 "" H 3450 4050 60  0000 C CNN
+F 2 "Connector_JST:JST_PH_B2B-PH-K_1x02_P2.00mm_Vertical" H 3450 4050 60  0001 C CNN
+F 3 "" H 3450 4050 60  0001 C CNN
 	1    3450 4050
 	-1   0    0    -1

Commit message: Simplify a bit.
Parts:
- J3: footprint Connector_PinHeader_2.54mm:PinHeader_2x05_P2.54mm_Vertical -> Connector_PinHeader_2.54mm:PinHeader_2x04_P2.54mm_Vertical; symbol Connector_Generic:Conn_02x05_Odd_Even -> Connector_Generic:Conn_02x04_Odd_Even
Connections:
- wire segments 163 -> 162
- no-connect marks 6 -> 7
Changed lines of the file:
@@
 	1    0    0    -1
 $EndComp
-Text Label 6400 900  2    50   ~ 0
+Text Label 6900 1100 0    50   ~ 0
 RTC_OUT
-Text Label 6400 1000 2    50   ~ 0
+Text Label 6900 1200 0    50   ~ 0
 RTC_TS
 $Comp
 L power:GND #PWR036
 U 1 1 5F7CED22
-P 7000 1250
-F 0 "#PWR036" H 7000 1000 50  0001 C CNN
-F 1 "GND" H 7000 1100 50  0000 C CNN
-F 2 "" H 7000 1250 60  0000 C CNN
-F 3 "" H 7000 1250 60  0000 C CNN
-	1    7000 1250
+P 6350 1250
+F 0 "#PWR036" H 6350 1000 50  0001 C CNN
+F 1 "GND" H 6350 1100 50  0000 C CNN
+F 2 "" H 6350 1250 60  0000 C CNN
+F 3 "" H 6350 1250 60  0000 C CNN
+	1    6350 1250
 	-1   0    0    -1
 $EndComp
@@
 Text Label 10600 2550 2    50   ~ 0
 DAC_OUT2
+Text Label 6900 900  0    50   ~ 0
+OCLK_LS
 Text Label 6900 1000 0    50   ~ 0
-OCLK_LS
-Text Label 6900 1100 0    50   ~ 0
 OCLK_M
 $Comp
@@
 $EndComp
 $Comp
-L Connector_Generic:Conn_02x05_Odd_Even J3
+L Connector_Generic:Conn_02x04_Odd_Even J3
 U 1 1 5FA992E3
 P 6600 1000
 F 0 "J3" H 6650 1417 50  0000 C CNN
 F 1 "CLOCKS" H 6650 1326 50  0000 C CNN
-F 2 "Connector_PinHeader_2.54mm:PinHeader_2x05_P2.54mm_Vertical" H 6600 1000 50  0001 C CNN
+F 2 "Connector_PinHeader_2.54mm:PinHeader_2x04_P2.54mm_Vertical" H 6600 1000 50  0001 C CNN
 F 3 "~" H 6600 1000 50  0001 C CNN
 	1    6600 1000
@@
 L power:VDD #PWR0113
 U 1 1 5FAB765C
-P 6300 750
-F 0 "#PWR0113" H 6300 600 50  0001 C CNN
-F 1 "VDD" H 6300 900 50  0000 C CNN
-F 2 "" H 6300 750 60  0000 C CNN
-F 3 "" H 6300 750 60  0000 C CNN
-	1    6300 750
+P 6300 900
+F 0 "#PWR0113" H 6300 750 50  0001 C CNN
+F 1 "VDD" H 6300 1050 50  0000 C CNN
+F 2 "" H 6300 900 60  0000 C CNN
+F 3 "" H 6300 900 60  0000 C CNN
+	1    6300 900
 	1    0    0    -1
 $EndComp
@@
 Wire Wire Line
 	2000 3050 2350 3050
-Text Label 6400 1200 2    50   ~ 0
-SWCLK_JTCK
-Text Label 8100 1100 2    50   ~ 0
-SWDIO_JTMS
-Text Label 8600 1100 0    50   ~ 0
-SWO_JTDO
-Wire Wire Line
-	6400 800  6300 800
-Wire Wire Line
-	6300 800  6300 750
-Wire Wire Line
-	6900 1200 7000 1200
-Wire Wire Line
-	7000 1200 7000 1250
-Text Label 6900 800  0    50   ~ 0
+Wire Wire Line
+	6400 900  6300 900
+Text Label 6400 1000 2    50   ~ 0
 EXTSCL
-Text Label 6900 900  0    50   ~ 0
+Text Label 6400 1100 2    50   ~ 0
 EXTSDA
 Text Label 3150 6800 0    50   ~ 0
@@
 Text Label 10650 1200 0    50   ~ 0
 RSTIN#
-Text Notes 5850 1350 0    40   ~ 0
+Text Notes 6500 1500 0    40   ~ 0
 Pin 7 was connected to PB15.
-NoConn ~ 6400 1100
 Text Label 10550 4700 0    50   ~ 0
 JTDI
@@
 	1    0    0    -1
 $EndComp
+NoConn ~ 8100 1100
+NoConn ~ 8600 1100
+Wire Wire Line
+	6400 1200 6350 1200
+Wire Wire Line
+	6350 1200 6350 1250
 $EndSCHEMATC

Commit message: Making more space.
Connections:
- net labels added: OTGFS_D+, OTGFS_D-, SPI2_CIPO, SPI2_COPI, SPI2_CS#
- net labels removed: OTG_FS_D+, OTG_FS_D-, SPI2_MISO, SPI2_MOSI, SPI2_SS#
Other:
- moved on the sheet: C1, C10, C11, C2, C5, C6, D1, D2, FB1, FB2, J1, J2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

Commit message: Fitting in bigger buttons and adding reset/boot circuit.
Parts:
- removed C7: 0.1uF, Capacitor_SMD:C_0603_1608Metric, symbol Device:C
- removed J5: SPI/USART, Connector_PinHeader_2.54mm:PinHeader_2x05_P2.54mm_Vertical, symbol Connector_Generic:Conn_02x05_Odd_Even
- removed Q1: BSS138BKS, Package_TO_SOT_SMD:SOT-363_SC-70-6, symbol @Engstad:BSS138BKS
- removed R2: 10k, Resistor_SMD:R_0603_1608Metric, symbol Device:R
- removed RN1: 10K, Resistor_SMD:R_Array_Concave_4x0603, symbol Device:R_Pack04_Split
- removed SW1: JUMPER_x2, Connector_PinHeader_2.54mm:PinHeader_2x03_P2.54mm_Vertical, symbol @Engstad:JUMPER_x2
- removed SW2: RST, engstad:tactile-switch-evpay-34x29mm, symbol @Engstad:SW_PUSH_NO
- removed SW3: USR, engstad:tactile-switch-evpay-34x29mm, symbol @Engstad:SW_PUSH_NO
- removed U3: APX823, Package_TO_SOT_SMD:SOT-23-5, symbol @Engstad:APX823
- added C20: 0.1uF, Capacitor_SMD:C_0603_1608Metric, symbol Device:C_Small
- added C21: 10uF/5%, Capacitor_SMD:C_0805_2012Metric, symbol Device:C
- added D3: 1N4148W, Diode_SMD:D_SOD-123, symbol Diode:1N4148W
- added J5: USART1, Connector_PinHeader_2.54mm:PinHeader_1x03_P2.54mm_Horizontal, symbol Connector_Generic:Conn_01x03
- added J8: SPI, Connector_PinHeader_2.54mm:PinHeader_2x03_P2.54mm_Vertical, symbol Connector_Generic:Conn_02x03_Odd_Even
- added Q2: DTC123JKA, Package_TO_SOT_SMD:SC-59, symbol Transistor_BJT:DTC123J
- added Q3: MMBFJ270, Package_TO_SOT_SMD:SOT-23, symbol Device:Q_PJFET_DSG
- added R6: 330K, Resistor_SMD:R_0603_1608Metric, symbol Device:R_Small_US
- added R7: 100R, Resistor_SMD:R_0603_1608Metric, symbol Device:R_Small_US
- added R8: 10K, Resistor_SMD:R_0603_1608Metric, symbol Device:R_Small_US
- added R9: 1M, Resistor_SMD:R_0603_1608Metric, symbol Device:R_Small_US
- added SW1, SW5: SW_PUSH_NO_ALT, engstad:TACTILE_SWITCH-TE-FSM4JSMAATR, symbol @Engstad:SW_PUSH_NO_ALT
- added SW4: JUMPER, Connector_PinHeader_2.54mm:PinHeader_1x03_P2.54mm_Vertical, symbol @Engstad:JUMPER
- C10: symbol Device:C -> Device:C_Small
- J3: footprint Connector_PinHeader_2.54mm:PinHeader_2x04_P2.54mm_Vertical -> Connector_PinHeader_2.54mm:PinHeader_2x03_P2.54mm_Vertical; symbol Connector_Generic:Conn_02x04_Odd_Even -> Connector_Generic:Conn_02x03_Odd_Even
- R1, R3, R4, R5: symbol Device:R -> Device:R_US
Connections:
- net labels added: RSTBTN
- net labels removed: +5V, BOOT_SEL, EXTSCL, EXTSDA, RSTIN#
- wire segments 162 -> 158
- no-connect marks 7 -> 4
Other:
- note removed: "Pin 7 was connected to PB15."
- note removed: "The APX823's manual reset line (~MR~) \nhas internal pullup of 60 kOhm.\n"
- moved on the sheet: C10, C4, C5, C6, FB2, NT1
