File: BetsyBoardBig.sch (KiCad schematic (older format))
At the start: 60 parts, among them J1 USB_B_Micro, J2 Micro_SD_Card, J3 CLOCKS, J4 USART3, J5 USART1, J6 I2C, J7 ANALOG, J8 SPI, P3 CORTEX-JTAG, P6 BATT, Q2 DTC123JKA, Q3 MMBFJ270, SW1 SW_PUSH_NO_ALT, SW4 JUMPER, SW5 SW_PUSH_NO_ALT, U1 TLV75733PDBVR‎, U2 USBLC6-2SC6, U4 STM32L486Rx-LQFP64, U5 IS25WP256D-xM, U6 74LVC1G3157, X1 XTAL, Y1 Crystal

Commit message: Additions due to single-button boot logic.
Parts:
- removed C20: 0.1uF, Capacitor_SMD:C_0603_1608Metric, symbol Device:C_Small
- removed C21: 10uF/5%, Capacitor_SMD:C_0805_2012Metric, symbol Device:C
- removed D3: 1N4148W, Diode_SMD:D_SOD-123, symbol Diode:1N4148W
- removed Q2: DTC123JKA, Package_TO_SOT_SMD:SC-59, symbol Transistor_BJT:DTC123J
- removed Q3: MMBFJ270, Package_TO_SOT_SMD:SOT-23, symbol Device:Q_PJFET_DSG
- removed R6: 330K, Resistor_SMD:R_0603_1608Metric, symbol Device:R_Small_US
- removed R7: 100R, Resistor_SMD:R_0603_1608Metric, symbol Device:R_Small_US
- removed R8: 10K, Resistor_SMD:R_0603_1608Metric, symbol Device:R_Small_US
- removed R9: 1M, Resistor_SMD:R_0603_1608Metric, symbol Device:R_Small_US
- added C11: 0.1uF, Capacitor_SMD:C_0603_1608Metric, symbol Device:C
- added C12: 10uF, Capacitor_SMD:C_0805_2012Metric, symbol Device:C
- added R1: 10K, Resistor_SMD:R_0603_1608Metric, symbol Device:R_US
- added R2: 1K, Resistor_SMD:R_0603_1608Metric, symbol Device:R_US
- added R3: 100K, Resistor_SMD:R_0603_1608Metric, symbol Device:R_US
- added TP1-RST#1, TP2-BOOT0: TestPoint_Probe, engstad:test-point-smd-5016, symbol Connector:TestPoint_Probe
- added U3: 74LVC3G14, Package_SO:SSOP-8_2.95x2.8mm_P0.65mm, symbol 74xGxx:74LVC3G14
- P2: renamed from P3; footprint engstad:conn-jtag-0.05 -> Connector_PinHeader_1.27mm:PinHeader_2x05_P1.27mm_Vertical
- SW2: renamed from SW5; value SW_PUSH_NO_ALT -> TE-FSM4J
- renumbered C3 to C1, C9 to C10, C4 to C13, C11 to C14, C12 to C15, C14 to C16, C15 to C17, C16 to C18, C17 to C19, C10 to C2, C19 to C20, C1 to C3, C2 to C4, C13 to C7, C18 to C8, C8 to C9, J3 to J1, J8 to J2, J1 to J3, J5 to J4, J6 to J5, J4 to J6, J2 to J8, P6 to P1, R5 to R4, R1 to R5, R3 to R6, R4 to R7, SW4 to SW1, SW1 to SW3, U6 to U5, U5 to U6
Connections:
- net labels added: ~MR
- net labels removed: RSTBTN
- wire segments 158 -> 156
- no-connect marks 4 -> 9
Other:
- note added: "A quick push of SW2 will cause ~RST~ to go low, resetting the uC.\n"
- note added: "Holding it for more than 0.3 s, will cause the uC to receive BOOT0 = 0,\nputting it in programming mode while begin reset. On release, the uC\nboots in programming mode, and 1.2 s after release, the uC goes back to \nBOOT0 = 1, which will take effect after the next reset."
- moved on the sheet: C10, C2, C5, C6, C9, FB2, NT1, Y1

Commit message: Prepare for second run.
Parts:
- removed J3: USB_B_Micro, engstad:usb-micro-b-amphenol-fci-10118194-oval, symbol Connector:USB_B_Micro
- removed J4: USART1, Connector_PinHeader_2.54mm:PinHeader_1x03_P2.54mm_Horizontal, symbol Connector_Generic:Conn_01x03
- added J3: USB_C_Receptacle_USB2.0, Connector_USB:USB_C_Receptacle_GCT_USB4085, symbol Connector:USB_C_Receptacle_USB2.0
- added J9: USART1, Connector_PinHeader_2.54mm:PinHeader_1x04_P2.54mm_Horizontal, symbol Connector_Generic:Conn_01x04
- added R8, R9: 5K1, Resistor_SMD:R_0603_1608Metric, symbol Device:R_US
- added TP2-BOOT1: TestPoint_Probe, engstad:pin-socket-1, symbol Connector:TestPoint_Probe
- TP1-NRST1: renamed from TP1-RST#1; footprint engstad:test-point-smd-5016 -> engstad:pin-socket-1
- TP2-BOOT0: footprint engstad:test-point-smd-5016 -> engstad:pin-socket-1
Connections:
- net labels added: CC1, CC2, ID+, ID-, USR_LED, ~JTRST
- net labels removed: LED_RED, OTGFS_D+, OTGFS_D-
- wire segments 156 -> 173
- no-connect marks 9 -> 10
Other:
- note added: "Note: ~JTRST~ only broken \nout as a test-point.\n"
- moved on the sheet: C5, C6, FB1, FB2, NT1, U2

Commit message: Use 4-pin QSPI NOR Flash card
Parts:
- removed U6: IS25WP256D-xM, Package_SO:SOIC-16W_7.5x10.3mm_P1.27mm, symbol Memory_Flash:IS25WP256D-xM
- added U6: IS25LP06D-xB, Package_SO:SOIC-8_5.275x5.275mm_P1.27mm, symbol @Engstad:IS25LP06D-xB
- J8: symbol Connector:Micro_SD_Card_Det1 -> @Engstad:SDMMC_Card_W_Det
Connections:
- no-connect marks 10 -> 8
Other:
- note added: "CX = 2*(CL - Cstray) = 2 * (12.5 - [2-5]) = [15 - 21] pF"
Changed lines of the file:
@@
 L power:GND #PWR054
 U 1 1 5F810F52
-P 3450 6000
-F 0 "#PWR054" H 3450 5750 50  0001 C CNN
-F 1 "GND" H 3450 5850 50  0000 C CNN
-F 2 "" H 3450 6000 60  0000 C CNN
-F 3 "" H 3450 6000 60  0000 C CNN
-	1    3450 6000
-	1    0    0    -1
-$EndComp
-Wire Wire Line
-	3350 5950 3450 5950
-Wire Wire Line
-	3450 5950 3450 6000
-$Comp
-L Connector:Micro_SD_Card_Det1 J8
+P 3400 5950
+F 0 "#PWR054" H 3400 5700 50  0001 C CNN
+F 1 "GND" H 3400 5800 50  0000 C CNN
+F 2 "" H 3400 5950 60  0000 C CNN
+F 3 "" H 3400 5950 60  0000 C CNN
+	1    3400 5950
+	1    0    0    -1
+$EndComp
+Wire Wire Line
+	3300 5900 3400 5900
+Wire Wire Line
+	3400 5900 3400 5950
+$Comp
+L @Engstad:SDMMC_Card_W_Det J8
 U 1 1 5F82D29C
-P 2550 5350
-F 0 "J8" H 2500 6067 50  0000 C CNN
-F 1 "Micro_SD_Card" H 2500 5976 50  0000 C CNN
-F 2 "engstad:Molex_PS_105162_001" H 3700 5650 50  0001 C CNN
-F 3 "https://www.molex.com/pdm_docs/sd/1051620001_sd.pdf" H 2550 5350 50  0001 C CNN
-F 4 "WM14405CT-ND" H 2550 5350 50  0001 C CNN "DigiKey#"
-	1    2550 5350
+P 2550 5450
+F 0 "J8" H 2500 6167 50  0000 C CNN
+F 1 "Micro_SD_Card" H 2500 6076 50  0000 C CNN
+F 2 "engstad:Molex_PS_105162_001" H 3700 5750 50  0001 C CNN
+F 3 "https://www.molex.com/pdm_docs/sd/1051620001_sd.pdf" H 2550 5450 50  0001 C CNN
+F 4 "WM14405CT-ND" H 2550 5450 50  0001 C CNN "DigiKey#"
+	1    2550 5450
 	1    0    0    -1
 $EndComp
@@
 	1    4250 7350
 	-1   0    0    1
-$EndComp
-$Comp
-L Memory_Flash:IS25WP256D-xM U6
-U 1 1 5F7865F4
-P 1400 7000
-F 0 "U6" H 1150 7450 50  0000 C CNN
-F 1 "IS25WP256D-xM" H 1750 6550 50  0000 C CNN
-F 2 "Package_SO:SOIC-16W_7.5x10.3mm_P1.27mm" H 1450 7600 50  0001 C CNN
-F 3 "http://www.issi.com/WW/pdf/IS25LP(WP)256D.pdf" H 1450 6500 50  0001 C CNN
-	1    1400 7000
-	1    0    0    -1
 $EndComp
 Connection ~ 800  5350
@@
 Text Label 900  6900 2    50   ~ 0
 QSPI_SCK
-NoConn ~ 1900 7100
 Text Label 900  7000 2    50   ~ 0
 QSPI_CS#
@@
 P 5300 3800
 F 0 "R3" V 5200 3850 50  0000 R CNN
-F 1 "100K" V 5400 3850 50  0000 R CNN
+F 1 "100K" V 5400 3900 50  0000 R CNN
 F 2 "Resistor_SMD:R_0603_1608Metric" H 5230 3708 30  0001 R CNN
 F 3 "" H 5300 3800 30  0000 C CNN
@@
 NoConn ~ 11900 2150
 NoConn ~ 8600 250
-NoConn ~ 6200 3400
 NoConn ~ 11450 1050
 Text Label 10550 5800 0    50   ~ 0
@@
 Text Notes 10450 1400 0    40   ~ 0
 Note: ~JTRST~ only broken \nout as a test-point.\n
+Text Notes 550  4400 0    50   ~ 0
+CX = 2*(CL - Cstray) = 2 * (12.5 - [2-5]) = [15 - 21] pF
+$Comp
+L @Engstad:IS25LP06D-xB U6
+U 1 1 60ABB36B
+P 1400 7000
+F 0 "U6" H 1050 7450 50  0000 C CNN
+F 1 "IS25LP06D-xB" H 1750 6550 50  0000 C CNN
+F 2 "Package_SO:SOIC-8_5.275x5.275mm_P1.27mm" H 1450 7600 50  0001 C CNN
+F 3 "http://www.issi.com/WW/pdf/IS25LP(WP)256D.pdf" H 1450 6500 50  0001 C CNN
+	1    1400 7000
+	1    0    0    -1
+$EndComp
 $EndSCHEMATC

Commit message: Latest work on big version
Parts:
- removed FB1: 220Ω@100MHz, Inductor_SMD:L_0805_2012Metric, symbol Device:Ferrite_Bead_Small
- added B1: BATT, engstad:Battery_Keystone_2894, symbol Device:Battery_Cell
- added C21, C22: 1uF, Capacitor_SMD:C_0805_2012Metric, symbol Device:C
- added D3: B130LAW, Diode_SMD:D_SOD-123, symbol Device:D_Schottky
- added F1: Polyfuse, Fuse:Fuse_0805_2012Metric, symbol Device:Polyfuse
- added Q1: FDN340P, Package_TO_SOT_SMD:SOT-23, symbol Transistor_FET:FDN340P
- added R10: 1K, Resistor_SMD:R_0603_1608Metric, symbol Device:R_US
- added R11: 100K, Resistor_SMD:R_0603_1608Metric, symbol Device:R_US
- added U7: MCP73831-2-OT, Package_TO_SOT_SMD:SOT-23-5, symbol Battery_Management:MCP73831-2-OT
- C12: value 10uF -> 1uF; footprint Capacitor_SMD:C_0805_2012Metric -> Capacitor_SMD:C_0603_1608Metric
- R3: value 100K -> 1M
- TP1: renamed from TP1-NRST1; footprint engstad:pin-socket-1 -> TestPoint:TestPoint_Pad_1.0x1.0mm
- TP2: renamed from TP2-BOOT0; footprint engstad:pin-socket-1 -> TestPoint:TestPoint_Pad_1.0x1.0mm
- renumbered TP2-BOOT1 to TP3
Connections:
- net labels added: PB8, PRG, VBUS_IN
- wire segments 173 -> 193
- no-connect marks 8 -> 6

Commit message: Getting ready for "final" big version.
Parts:
- removed C13: 0.1uF, Capacitor_SMD:C_0603_1608Metric, symbol Device:C
- removed R5: 1K, Resistor_SMD:R_0603_1608Metric, symbol Device:R_US
- added D4: RED, LED_SMD:LED_0603_1608Metric, symbol Device:LED
- D1: value RED -> BLUE
- J7: footprint Connector_PinHeader_2.54mm:PinHeader_1x10_P2.54mm_Horizontal -> Connector_PinHeader_2.54mm:PinHeader_2x06_P2.54mm_Horizontal; symbol Connector_Generic:Conn_01x10 -> Connector_Generic:Conn_02x06_Odd_Even
- R4: value 10K -> 470
- R7: value 180 -> 1K
Connections:
- net labels added: COIN+, STAT, VBATT, VCOIN
- net labels removed: USR_BTN, VBAT_IN
- wire segments 193 -> 196
- no-connect marks 6 -> 4

Commit message: Thsi too.
Parts:
- added C13: 0.1uF, Capacitor_SMD:C_0603_1608Metric, symbol Device:C_Small
- added R12: 1K, Resistor_SMD:R_0603_1608Metric, symbol Device:R_US
- added R5: 10K, Resistor_SMD:R_0603_1608Metric, symbol Device:R_US
Connections:
- wire segments 196 -> 201
Other:
- note added: "D"
- note added: "G"
- note added: "In order for switch to turn on, VIN = Vs >= Vg + Vth = VBUS + Vth.\nWith battery powered, the body diode makes Vs = 4.2V - 0.7V = 3.5V,\nfor a moment. Then 3.5V >= 0V + 2V, so the switch turns on, bringing \nVIN to 4.2V - Rds * Id. \n\nWhen VBATT is 0V, and VBUS = 5V, then \nVIN = 5V - 0..3V = 4.7V < VBUS.+ Vth = 5V + 2V = 7V, \nso the switch is off, and VIN = VBUS - 0.3V"
- note added: "S"
- moved on the sheet: D4
Changed lines of the file:
@@
 U 1 1 5603811A
 P 5750 1050
-F 0 "C2" H 5550 1150 50  0000 L CNN
-F 1 "0.1uF" H 5500 950 50  0000 L CNN
+F 0 "C2" H 5550 1100 50  0000 L CNN
+F 1 "0.1uF" H 5450 1000 50  0000 L CNN
 F 2 "Capacitor_SMD:C_0603_1608Metric" H 5788 900 30  0001 C CNN
 F 3 "" H 5750 1050 60  0000 C CNN
@@
 	0    -1   -1   0
 $EndComp
-Wire Wire Line
-	5450 1700 5550 1700
 $Comp
 L @Engstad:SW_PUSH_NO_ALT SW3
 U 1 1 60310734
-P 5450 1900
-F 0 "SW3" V 5450 1854 60  0000 R CNN
-F 1 "SW_PUSH_NO_ALT" H 5450 2058 60  0001 C CNN
-F 2 "engstad:TACTILE_SWITCH-TE-FSM4JSMAATR" H 5450 2164 60  0001 C CNN
-F 3 "https://www.mouser.com/datasheet/2/418/1/NG_CD_2-1437565-7_V-663781.pdf" H 5450 2058 60  0001 C CNN
-	1    5450 1900
+P 5450 2000
+F 0 "SW3" V 5450 1954 60  0000 R CNN
+F 1 "SW_PUSH_NO_ALT" H 5450 2158 60  0001 C CNN
+F 2 "engstad:TACTILE_SWITCH-TE-FSM4JSMAATR" H 5450 2264 60  0001 C CNN
+F 3 "https://www.mouser.com/datasheet/2/418/1/NG_CD_2-1437565-7_V-663781.pdf" H 5450 2158 60  0001 C CNN
+	1    5450 2000
 	0    -1   -1   0
 $EndComp
 Wire Wire Line
-	5450 1750 5450 1700
+	5450 1850 5450 1800
 $Comp
 L power:GND #PWR047
 U 1 1 5F85A6F2
-P 5450 2050
-F 0 "#PWR047" H 5450 1800 50  0001 C CNN
-F 1 "GND" H 5450 1900 50  0000 C CNN
-F 2 "" H 5450 2050 60  0000 C CNN
-F 3 "" H 5450 2050 60  0000 C CNN
-	1    5450 2050
-	1    0    0    -1
-$EndComp
-Text Label 5550 1700 0    50   ~ 0
+P 5450 2150
+F 0 "#PWR047" H 5450 1900 50  0001 C CNN
+F 1 "GND" H 5450 2000 50  0000 C CNN
+F 2 "" H 5450 2150 60  0000 C CNN
+F 3 "" H 5450 2150 60  0000 C CNN
+	1    5450 2150
+	1    0    0    -1
+$EndComp
+Text Label 6200 1800 0    50   ~ 0
 USR_SW
 Text Label 5500 -400 0    50   ~ 0
@@
 L Device:LED D4
 U 1 1 60D0502B
-P 4750 5300
-F 0 "D4" V 4796 5192 50  0000 R CNN
-F 1 "RED" V 4704 5192 50  0000 R CNN
-F 2 "LED_SMD:LED_0603_1608Metric" H 4750 5300 60  0001 C CNN
-F 3 "" H 4750 5300 60  0000 C CNN
-	1    4750 5300
+P 4800 5300
+F 0 "D4" V 4846 5192 50  0000 R CNN
+F 1 "RED" V 4754 5192 50  0000 R CNN
+F 2 "LED_SMD:LED_0603_1608Metric" H 4800 5300 60  0001 C CNN
+F 3 "" H 4800 5300 60  0000 C CNN
+	1    4800 5300
 	0    -1   -1   0
 $EndComp
@@
 L Device:R_US R4
 U 1 1 60D1EC17
-P 4750 5750
-F 0 "R4" H 4820 5826 50  0000 L CNN
-F 1 "470" H 4820 5734 50  0000 L CNN
-F 2 "Resistor_SMD:R_0603_1608Metric" H 4820 5658 30  0001 L CNN
-F 3 "" H 4750 5750 30  0000 C CNN
-	1    4750 5750
-	1    0    0    -1
-$EndComp
-Wire Wire Line
-	4750 4900 4750 5150
-Wire Wire Line
-	4750 5450 4750 5600
-Wire Wire Line
-	4750 5900 4750 6050
-Wire Wire Line
-	4750 6050 4900 6050
-Text Label 4900 6050 0    50   ~ 0
+P 4800 5750
+F 0 "R4" H 4870 5826 50  0000 L CNN
+F 1 "470" H 4870 5734 50  0000 L CNN
+F 2 "Resistor_SMD:R_0603_1608Metric" H 4870 5658 30  0001 L CNN
+F 3 "" H 4800 5750 30  0000 C CNN
+	1    4800 5750
+	1    0    0    -1
+$EndComp
+Wire Wire Line
+	4800 4900 4800 5150
+Wire Wire Line
+	4800 5450 4800 5600
+Wire Wire Line
+	4800 5900 4800 6050
+Wire Wire Line
+	4800 6050 4950 6050
+Text Label 4950 6050 0    50   ~ 0
 STAT
 Wire Wire Line
@@
 Wire Wire Line
 	11150 2400 10950 2400
-Text Label 4750 4900 0    50   ~ 0
+Text Label 4800 4900 0    50   ~ 0
 VIN
 Text Label 4950 1000 0    50   ~ 0
 COIN+
+Text Notes 5900 -1250 0    50   ~ 0
+G
+Text Notes 6250 -1300 0    50   ~ 0
+S
+Text Notes 6250 -950 0    50   ~ 0
+D
+Text Notes 5750 -2150 0    50   ~ 0
+In order for switch to turn on, VIN = Vs >= Vg + Vth = VBUS + Vth.\nWith battery powered, the body diode makes Vs = 4.2V - 0.7V = 3.5V,\nfor a moment. Then 3.5V >= 0V + 2V, so the switch turns on, bringing \nVIN to 4.2V - Rds * Id. \n\nWhen VBATT is 0V, and VBUS = 5V, then \nVIN = 5V - 0..3V = 4.7V < VBUS.+ Vth = 5V + 2V = 7V, \nso the switch is off, and VIN = VBUS - 0.3V
+$Comp
+L Device:C_Small C13
+U 1 1 6103B013
+P 5950 2000
+F 0 "C13" H 5750 2050 50  0000 L CNN
+F 1 "0.1uF" H 5650 1950 50  0000 L CNN
+F 2 "Capacitor_SMD:C_0603_1608Metric" H 5988 1850 30  0001 C CNN
+F 3 "" H 5950 2000 60  0000 C CNN
+	1    5950 2000
+	-1   0    0    -1
+$EndComp
+$Comp
+L power:GND #PWR0102
+U 1 1 6103C2E5
+P 5950 2150
+F 0 "#PWR0102" H 5950 1900 50  0001 C CNN
+F 1 "GND" H 5950 2000 50  0000 C CNN
+F 2 "" H 5950 2150 60  0000 C CNN
+F 3 "" H 5950 2150 60  0000 C CNN
+	1    5950 2150
+	1    0    0    -1
+$EndComp
+Wire Wire Line
+	5950 2100 5950 2150
+Wire Wire Line
+	5450 1800 5550 1800
+Wire Wire Line
+	5950 1900 5950 1800
+Connection ~ 5950 1800
+Wire Wire Line
+	5950 1800 6200 1800
+$Comp
+L Device:R_US R12
+U 1 1 61083B55
+P 5700 1800
+F 0 "R12" V 5600 1850 50  0000 R CNN
+F 1 "1K" V 5800 1850 50  0000 R CNN
+F 2 "Resistor_SMD:R_0603_1608Metric" H 5630 1708 30  0001 R CNN
+F 3 "" H 5700 1800 30  0000 C CNN
+	1    5700 1800
+	0    1    1    0
+$EndComp
+Wire Wire Line
+	5850 1800 5950 1800
+$Comp
+L Device:R_US R5
+U 1 1 61085886
+P 5450 1600
+F 0 "R5" H 5380 1676 50  0000 R CNN
+F 1 "10K" H 5380 1584 50  0000 R CNN
+F 2 "Resistor_SMD:R_0603_1608Metric" H 5380 1508 30  0001 R CNN
+F 3 "" H 5450 1600 30  0000 C CNN
+	1    5450 1600
+	-1   0    0    -1
+$EndComp
+Wire Wire Line
+	5450 1750 5450 1800
+Connection ~ 5450 1800
+$Comp
+L power:VDD #PWR0105
+U 1 1 61092D9C
+P 5450 1450
+F 0 "#PWR0105" H 5450 1300 50  0001 C CNN
+F 1 "VDD" H 5450 1600 50  0000 C CNN
+F 2 "" H 5450 1450 60  0000 C CNN
+F 3 "" H 5450 1450 60  0000 C CNN
+	1    5450 1450
+	1    0    0    -1
+$EndComp
 $EndSCHEMATC

Commit message: Save from old computer.
Parts:
- added TP4: TestPoint_Probe, TestPoint:TestPoint_Pad_1.0x1.0mm, symbol Connector:TestPoint_Probe
Connections:
- net labels added: SW3
- wire segments 201 -> 202
Other:
- moved on the sheet: C13
Changed lines of the file:
@@
-	0    -1   -1   0
-$EndComp
-$Comp
-L @Engstad:SW_PUSH_NO_ALT SW3
-U 1 1 60310734
-P 5450 2000
-F 0 "SW3" V 5450 1954 60  0000 R CNN
-F 1 "SW_PUSH_NO_ALT" H 5450 2158 60  0001 C CNN
-F 2 "engstad:TACTILE_SWITCH-TE-FSM4JSMAATR" H 5450 2264 60  0001 C CNN
-F 3 "https://www.mouser.com/datasheet/2/418/1/NG_CD_2-1437565-7_V-663781.pdf" H 5450 2158 60  0001 C CNN
-	1    5450 2000
 	0    -1   -1   0
 $EndComp
 Wire Wire Line
-	5450 1850 5450 1800
+	5450 1800 5450 1750
 $Comp
 L power:GND #PWR047
 U 1 1 5F85A6F2
-P 5450 2150
-F 0 "#PWR047" H 5450 1900 50  0001 C CNN
-F 1 "GND" H 5450 2000 50  0000 C CNN
-F 2 "" H 5450 2150 60  0000 C CNN
-F 3 "" H 5450 2150 60  0000 C CNN
-	1    5450 2150
+P 5450 2100
+F 0 "#PWR047" H 5450 1850 50  0001 C CNN
+F 1 "GND" H 5450 1950 50  0000 C CNN
+F 2 "" H 5450 2100 60  0000 C CNN
+F 3 "" H 5450 2100 60  0000 C CNN
+	1    5450 2100
 	1    0    0    -1
 $EndComp
-Text Label 6200 1800 0    50   ~ 0
+Text Label 6200 1750 0    50   ~ 0
 USR_SW
 Text Label 5500 -400 0    50   ~ 0
@@
 L Device:C_Small C13
 U 1 1 6103B013
-P 5950 2000
-F 0 "C13" H 5750 2050 50  0000 L CNN
-F 1 "0.1uF" H 5650 1950 50  0000 L CNN
-F 2 "Capacitor_SMD:C_0603_1608Metric" H 5988 1850 30  0001 C CNN
-F 3 "" H 5950 2000 60  0000 C CNN
-	1    5950 2000
+P 6050 1950
+F 0 "C13" H 5850 2000 50  0000 L CNN
+F 1 "0.1uF" H 5750 1900 50  0000 L CNN
+F 2 "Capacitor_SMD:C_0603_1608Metric" H 6088 1800 30  0001 C CNN
+F 3 "" H 6050 1950 60  0000 C CNN
+	1    6050 1950
 	-1   0    0    -1
 $EndComp
@@
 L power:GND #PWR0102
 U 1 1 6103C2E5
-P 5950 2150
-F 0 "#PWR0102" H 5950 1900 50  0001 C CNN
-F 1 "GND" H 5950 2000 50  0000 C CNN
-F 2 "" H 5950 2150 60  0000 C CNN
-F 3 "" H 5950 2150 60  0000 C CNN
-	1    5950 2150
+P 6050 2100
+F 0 "#PWR0102" H 6050 1850 50  0001 C CNN
+F 1 "GND" H 6050 1950 50  0000 C CNN
+F 2 "" H 6050 2100 60  0000 C CNN
+F 3 "" H 6050 2100 60  0000 C CNN
+	1    6050 2100
 	1    0    0    -1
 $EndComp
 Wire Wire Line
-	5950 2100 5950 2150
+	6050 2050 6050 2100
 Wire Wire Line
-	5450 1800 5550 1800
+	5450 1750 5650 1750
 Wire Wire Line
-	5950 1900 5950 1800
-Connection ~ 5950 1800
+	6050 1850 6050 1750
+Connection ~ 6050 1750
 Wire Wire Line
-	5950 1800 6200 1800
+	6050 1750 6200 1750
 $Comp
 L Device:R_US R12
 U 1 1 61083B55
-P 5700 1800
-F 0 "R12" V 5600 1850 50  0000 R CNN
-F 1 "1K" V 5800 1850 50  0000 R CNN
-F 2 "Resistor_SMD:R_0603_1608Metric" H 5630 1708 30  0001 R CNN
-F 3 "" H 5700 1800 30  0000 C CNN
-	1    5700 1800
+P 5800 1750
+F 0 "R12" V 5700 1800 50  0000 R CNN
+F 1 "1K" V 5900 1800 50  0000 R CNN
+F 2 "Resistor_SMD:R_0603_1608Metric" H 5730 1658 30  0001 R CNN
+F 3 "" H 5800 1750 30  0000 C CNN
+	1    5800 1750
 	0    1    1    0
 $EndComp
 Wire Wire Line
-	5850 1800 5950 1800
+	5950 1750 6050 1750
 $Comp
 L Device:R_US R5
 U 1 1 61085886
-P 5450 1600
-F 0 "R5" H 5380 1676 50  0000 R CNN
-F 1 "10K" H 5380 1584 50  0000 R CNN
-F 2 "Resistor_SMD:R_0603_1608Metric" H 5380 1508 30  0001 R CNN
-F 3 "" H 5450 1600 30  0000 C CNN
-	1    5450 1600
+P 6050 1550
+F 0 "R5" H 5980 1626 50  0000 R CNN
+F 1 "10K" H 5980 1534 50  0000 R CNN
+F 2 "Resistor_SMD:R_0603_1608Metric" H 5980 1458 30  0001 R CNN
+F 3 "" H 6050 1550 30  0000 C CNN
+	1    6050 1550
 	-1   0    0    -1
 $EndComp
-Wire Wire Line
-	5450 1750 5450 1800
-Connection ~ 5450 1800
 $Comp
 L power:VDD #PWR0105
 U 1 1 61092D9C
-P 5450 1450
-F 0 "#PWR0105" H 5450 1300 50  0001 C CNN
-F 1 "VDD" H 5450 1600 50  0000 C CNN
-F 2 "" H 5450 1450 60  0000 C CNN
-F 3 "" H 5450 1450 60  0000 C CNN
-	1    5450 1450
+P 6050 1400
+F 0 "#PWR0105" H 6050 1250 50  0001 C CNN
+F 1 "VDD" H 6050 1550 50  0000 C CNN
+F 2 "" H 6050 1400 60  0000 C CNN
+F 3 "" H 6050 1400 60  0000 C CNN
+	1    6050 1400
 	1    0    0    -1
 $EndComp
+Wire Wire Line
+	6050 1700 6050 1750
+Text Label 5450 1750 0    50   ~ 0
+SW3
+$Comp
+L @Engstad:SW_PUSH_NO_ALT SW3
+U 1 1 60310734
+P 5450 1950
+F 0 "SW3" V 5450 1904 60  0000 R CNN
+F 1 "SW_PUSH_NO_ALT" H 5450 2108 60  0001 C CNN
+F 2 "engstad:TACTILE_SWITCH-TE-FSM4JSMAATR" H 5450 2214 60  0001 C CNN
+F 3 "https://www.mouser.com/datasheet/2/418/1/NG_CD_2-1437565-7_V-663781.pdf" H 5450 2108 60  0001 C CNN
+	1    5450 1950
+	0    -1   -1   0
+$EndComp
+$Comp
+L Connector:TestPoint_Probe TP4
+U 1 1 60CA436A
+P 9050 2400
+F 0 "TP4" H 9203 2501 50  0000 L CNN
+F 1 "TestPoint_Probe" H 9203 2410 50  0001 L CNN
+F 2 "TestPoint:TestPoint_Pad_1.0x1.0mm" H 9250 2400 50  0001 C CNN
+F 3 "~" H 9250 2400 50  0001 C CNN
+	1    9050 2400
+	1    0    0    -1
+$EndComp
+Text Label 9000 2400 2    50   ~ 0
+BOOT0
+Wire Wire Line
+	9000 2400 9050 2400
 $EndSCHEMATC
